File: Platinen/520-WS2811_Extender/WS2811_Extender_V1.1.brd (EAGLE design)
At the start: 49.6 x 16 mm, 26 parts, among them IC1 ULN2003AN, J1 Out2, J2 Out3, J4 Out1, U2R TINY45-20-DIP, U3H WS2811 SOT-8

Commit message: Ver.:1.1
Other:
- board text added: "27.07.20"
- board text removed: "26.07.20"
Changed lines of the file:
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@@
 <grid distance="50" unitdist="mil" unit="mil" style="lines" multiple="1" display="yes" altdistance="6.25" altunitdist="mil" altunit="mil"/>
 <layers>
-<layer number="1" name="Top" color="4" fill="1" visible="no" active="yes"/>
+<layer number="1" name="Top" color="4" fill="1" visible="yes" active="yes"/>
 <layer number="16" name="Bottom" color="1" fill="1" visible="no" active="yes"/>
 <layer number="17" name="Pads" color="2" fill="1" visible="yes" active="yes"/>
@@
 <layer number="19" name="Unrouted" color="6" fill="1" visible="yes" active="yes"/>
 <layer number="20" name="Dimension" color="24" fill="1" visible="yes" active="yes"/>
-<layer number="21" name="tPlace" color="7" fill="1" visible="no" active="yes"/>
-<layer number="22" name="bPlace" color="7" fill="1" visible="yes" active="yes"/>
-<layer number="23" name="tOrigins" color="15" fill="1" visible="no" active="yes"/>
-<layer number="24" name="bOrigins" color="15" fill="1" visible="yes" active="yes"/>
-<layer number="25" name="tNames" color="7" fill="1" visible="no" active="yes"/>
-<layer number="26" name="bNames" color="7" fill="1" visible="yes" active="yes"/>
+<layer number="21" name="tPlace" color="7" fill="1" visible="yes" active="yes"/>
+<layer number="22" name="bPlace" color="7" fill="1" visible="no" active="yes"/>
+<layer number="23" name="tOrigins" color="15" fill="1" visible="yes" active="yes"/>
+<layer number="24" name="bOrigins" color="15" fill="1" visible="no" active="yes"/>
+<layer number="25" name="tNames" color="7" fill="1" visible="yes" active="yes"/>
+<layer number="26" name="bNames" color="7" fill="1" visible="no" active="yes"/>
 <layer number="27" name="tValues" color="7" fill="1" visible="no" active="yes"/>
 <layer number="28" name="bValues" color="7" fill="1" visible="no" active="yes"/>
@@
 <layer number="37" name="tTest" color="7" fill="1" visible="no" active="yes"/>
 <layer number="38" name="bTest" color="7" fill="1" visible="no" active="yes"/>
-<layer number="39" name="tKeepout" color="4" fill="11" visible="no" active="yes"/>
-<layer number="40" name="bKeepout" color="1" fill="11" visible="yes" active="yes"/>
-<layer number="41" name="tRestrict" color="4" fill="10" visible="no" active="yes"/>
-<layer number="42" name="bRestrict" color="1" fill="10" visible="yes" active="yes"/>
+<layer number="39" name="tKeepout" color="4" fill="11" visible="yes" active="yes"/>
+<layer number="40" name="bKeepout" color="1" fill="11" visible="no" active="yes"/>
+<layer number="41" name="tRestrict" color="4" fill="10" visible="yes" active="yes"/>
+<layer number="42" name="bRestrict" color="1" fill="10" visible="no" active="yes"/>
 <layer number="43" name="vRestrict" color="2" fill="10" visible="no" active="yes"/>
 <layer number="44" name="Drills" color="7" fill="1" visible="no" active="yes"/>
@@
 <layer number="49" name="Reference" color="7" fill="1" visible="no" active="yes"/>
 <layer number="50" name="dxf" color="7" fill="1" visible="no" active="no"/>
-<layer number="51" name="tDocu" color="7" fill="1" visible="no" active="yes"/>
+<layer number="51" name="tDocu" color="7" fill="1" visible="yes" active="yes"/>
 <layer number="52" name="bDocu" color="7" fill="1" visible="yes" active="yes"/>
 <layer number="53" name="tGND_GNDA" color="7" fill="9" visible="no" active="no"/>
@@
 <wire x1="50" y1="16.055" x2="0.4" y2="16.055" width="0" layer="20"/>
 <wire x1="0.4" y1="16.055" x2="0.4" y2="0.065" width="0" layer="20"/>
-<text x="46.2915" y="0.47625" size="0.8636" layer="52" rot="MR0">26.07.20</text>
+<text x="46.2915" y="0.47625" size="0.8636" layer="52" rot="MR0">27.07.20</text>
 <text x="40.1828" y="11.3284" size="1.27" layer="52" rot="MR0">WS2811 Extender</text>
 <text x="42.8752" y="12.8016" size="0.8128" layer="52" rot="MR180">400 mA</text>
@@
 <text x="1.25095" y="7.6581" size="0.7112" layer="52" rot="MR270">GND</text>
 <text x="1.25095" y="9.9695" size="0.7112" layer="52" rot="MR270">Out</text>
-<dimension x1="0.4" y1="0.065" x2="50" y2="0.065" x3="25.2" y3="-3.81" textsize="1.778" layer="48"/>
-<dimension x1="0.4" y1="16.055" x2="0.4" y2="0.065" x3="-0.889" y3="8.06" textsize="1.778" layer="48"/>
 <wire x1="50" y1="16.055" x2="0.4" y2="16.055" width="0.1524" layer="22"/>
 <wire x1="0.4" y1="16.055" x2="0.4" y2="0.065" width="0.1524" layer="22"/>
@@
 <text x="1.25095" y="12.7381" size="0.7112" layer="52" rot="MR270">GND</text>
 <text x="1.25095" y="15.5956" size="0.7112" layer="52" rot="MR270">5/12V</text>
+<wire x1="11.27125" y1="14.2875" x2="11.27125" y2="18.57375" width="1.27" layer="51"/>
+<wire x1="13.81125" y1="14.2875" x2="13.81125" y2="18.57375" width="1.27" layer="51"/>
+<wire x1="16.35125" y1="14.2875" x2="16.35125" y2="18.57375" width="1.27" layer="51"/>
+<wire x1="18.89125" y1="14.2875" x2="18.89125" y2="18.57375" width="1.27" layer="51"/>
+<wire x1="21.43125" y1="14.2875" x2="21.43125" y2="18.57375" width="1.27" layer="51"/>
+<wire x1="23.97125" y1="14.2875" x2="23.97125" y2="18.57375" width="1.27" layer="51"/>
+<wire x1="11.27125" y1="14.2875" x2="11.27125" y2="18.57375" width="1.27" layer="52"/>
+<wire x1="13.81125" y1="14.2875" x2="13.81125" y2="18.57375" width="1.27" layer="52"/>
+<wire x1="16.35125" y1="14.2875" x2="16.35125" y2="18.57375" width="1.27" layer="52"/>
+<wire x1="18.89125" y1="14.2875" x2="18.89125" y2="18.57375" width="1.27" layer="52"/>
+<wire x1="21.43125" y1="14.2875" x2="21.43125" y2="18.57375" width="1.27" layer="52"/>
+<wire x1="23.97125" y1="14.2875" x2="23.97125" y2="18.57375" width="1.27" layer="52"/>
 </plain>
 <attributes>
@@
 <wire x1="18.89125" y1="5.332815625" x2="18.2118" y2="5.9152" width="0.5588" layer="16"/>
 <contactref element="C1R" pad="2"/>
-<wire x1="19.9136" y1="3.1115" x2="22.36351875" y2="3.1115" width="0.508" layer="16"/>
-<wire x1="19.9136" y1="3.1115" x2="19.9136" y2="3.16865" width="0.508" layer="16"/>
-<wire x1="19.9136" y1="3.16865" x2="18.89125" y2="4.191" width="0.508" layer="16"/>
 <wire x1="18.89125" y1="4.191" x2="18.40865" y2="3.7084" width="0.5588" layer="16"/>
 <wire x1="18.40865" y1="3.7084" x2="18.40865" y2="3.599575" width="0.5588" layer="16"/>
@@
 <wire x1="26.51125" y1="1.905" x2="25.7175" y2="1.905" width="0.5842" layer="16"/>
 <wire x1="25.7175" y1="1.905" x2="23.97125" y2="1.905" width="0.5842" layer="16"/>
-<wire x1="22.36351875" y1="3.1115" x2="23.57001875" y2="1.905" width="0.508" layer="16"/>
-<wire x1="23.57001875" y1="1.905" x2="23.97125" y2="1.905" width="0.5842" layer="16"/>
 <wire x1="25.71115" y1="4.064" x2="25.71115" y2="1.91135" width="0.5842" layer="16"/>
 <wire x1="25.71115" y1="1.91135" x2="25.7175" y2="1.905" width="0.5842" layer="16"/>
@@
 <wire x1="2.5527" y1="11.4935" x2="4.58460625" y2="11.4935" width="0.5842" layer="1"/>
 <wire x1="4.58460625" y1="11.4935" x2="5.91810625" y2="10.16" width="0.5842" layer="1"/>
+<wire x1="19.95975" y1="3.1225" x2="18.89125" y2="4.191" width="0.3302" layer="16"/>
+<wire x1="23.6802625" y1="1.905" x2="22.4627625" y2="3.1225" width="0.3302" layer="16"/>
+<wire x1="22.4627625" y1="3.1225" x2="19.95975" y2="3.1225" width="0.3302" layer="16"/>
+<wire x1="23.97125" y1="1.905" x2="23.6802625" y2="1.905" width="0.3302" layer="16"/>
 </signal>
 <signal name="N$1">
@@
 <wire x1="14.92885" y1="3.72806875" x2="14.92885" y2="4.34913125" width="0.4064" layer="16"/>
 <wire x1="14.92885" y1="4.34913125" x2="16.9562" y2="6.37648125" width="0.4064" layer="16"/>
-<wire x1="22.5397" y1="2.9464" x2="21.59" y2="3.8961" width="0.254" layer="1"/>
 <polygon width="0.1524" layer="1">
 <vertex x="12.7" y="15.24"/>
@@
 <via x="27.07995" y="3.81" extent="1-16" drill="0.35"/>
 <wire x1="27.07995" y1="3.81" x2="27.07995" y2="4.51621875" width="0.254" layer="1"/>
-<wire x1="27.07995" y1="3.81" x2="26.21635" y2="2.9464" width="0.254" layer="1"/>
-<wire x1="26.21635" y1="2.9464" x2="22.5397" y2="2.9464" width="0.254" layer="1"/>
 <contactref element="JP1" pad="1"/>
 <wire x1="27.07995" y1="4.51621875" x2="26.2001" y2="5.39606875" width="0.254" layer="1"/>
@@
 <wire x1="26.61565" y1="8.9972" x2="26.61565" y2="7.71948125" width="0.254" layer="1"/>
 <wire x1="26.61565" y1="7.71948125" x2="26.2001" y2="7.30393125" width="0.254" layer="1"/>
+<wire x1="22.70821875" y1="2.9464" x2="23.63408125" y2="2.9464" width="0.254" layer="1"/>
+<wire x1="24.59355" y1="4.52693125" x2="25.24821875" y2="5.1816" width="0.254" layer="1"/>
+<wire x1="25.24821875" y1="5.1816" x2="25.98563125" y2="5.1816" width="0.254" layer="1"/>
+<wire x1="25.98563125" y1="5.1816" x2="26.2001" y2="5.39606875" width="0.254" layer="1"/>
+<wire x1="21.59" y1="3.8961" x2="21.75851875" y2="3.8961" width="0.254" layer="1"/>
+<wire x1="24.59355" y1="3.90586875" x2="24.59355" y2="4.52693125" width="0.254" layer="1"/>
+<wire x1="21.75851875" y1="3.8961" x2="22.70821875" y2="2.9464" width="0.254" layer="1"/>
+<wire x1="23.63408125" y1="2.9464" x2="24.59355" y2="3.90586875" width="0.254" layer="1"/>
 </signal>
 <signal name="N$4">
