File: Platinen/520-WS2811_Extender/WS2811_Extender_V1.1_X12.brd (EAGLE design)
At the start: 100 x 100 mm, 312 parts, among them IC1 ULN2003AN, IC10 ULN2003AN, IC11 ULN2003AN, IC12 ULN2003AN, IC2 ULN2003AN, IC3 ULN2003AN, IC4 ULN2003AN, IC5 ULN2003AN, IC6 ULN2003AN, IC7 ULN2003AN, IC8 ULN2003AN, IC9 ULN2003AN, J1 Out2, J10 Out1, J11 Out2, J12 Out3, J13 Out1, J14 Out2, J15 Out3, J16 Out1, J17 Out2, J18 Out3, J19 Out1, J2 Out3, J20 Out2, J21 Out3, J22 Out1, J23 Out2, J24 Out3, J25 Out1, J26 Out2, J27 Out3, J28 Out1, J29 Out2, J3 Out1, J30 Out3, J31 Out1, J32 Out2, J33 Out3, J34 Out1, J35 Out2, J36 Out3, J4 Out1, J5 Out2, J6 Out3, J7 Out1, J8 Out2, J9 Out3, U2R TINY45-20-DIP, U2R1 TINY45-20-DIP, U2R10 TINY45-20-DIP, U2R11 TINY45-20-DIP, U2R2 TINY45-20-DIP, U2R3 TINY45-20-DIP, U2R4 TINY45-20-DIP, U2R5 TINY45-20-DIP, U2R6 TINY45-20-DIP, U2R7 TINY45-20-DIP, U2R8 TINY45-20-DIP, U2R9 TINY45-20-DIP, U3H WS2811 SOT-8, U3H1 WS2811 SOT-8, U3H10 WS2811 SOT-8, U3H11 WS2811 SOT-8, U3H2 WS2811 SOT-8, U3H3 WS2811 SOT-8, U3H4 WS2811 SOT-8, U3H5 WS2811 SOT-8, U3H6 WS2811 SOT-8, U3H7 WS2811 SOT-8, U3H8 WS2811 SOT-8, U3H9 WS2811 SOT-8

Commit message: Ver.:1.1
Parts:
- moved 6=12V10 2.54 mm to (81.1, 103.8)
- moved 6=12V2 2.54 mm to (30.7, 70.2)
- moved 6=12V4 2.54 mm to (30.7, 103.8)
- moved 6=12V8 2.54 mm to (81.1, 70.2)
- moved 6=5V11 2.54 mm to (81.4, 109.2)
- moved 6=5V3 2.54 mm to (31.0, 75.6)
- moved 6=5V5 2.54 mm to (31.0, 109.2)
- moved 6=5V9 2.54 mm to (81.4, 75.6)
- moved C1H11 2.54 mm to (94.6, 113.9)
- moved C1H3 2.54 mm to (44.2, 80.3)
- moved C1H5 2.54 mm to (44.2, 113.9)
- moved C1H9 2.54 mm to (94.6, 80.3)
- moved C1R1 2.54 mm to (50.4, 43.5)
- moved C1R11 2.54 mm to (100.8, 110.7)
- moved C1R3 2.54 mm to (50.4, 77.1)
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Routing:
- net S$89: track 0.00 -> 4.29 mm
- net S$88: track 0.00 -> 4.29 mm
- net S$87: track 0.00 -> 4.29 mm
- net S$86: track 0.00 -> 4.29 mm
- net S$85: track 0.00 -> 4.29 mm
- net S$84: track 0.00 -> 4.29 mm
- net S$36: track 0.00 -> 4.29 mm
- net S$35: track 0.00 -> 4.29 mm
- net S$34: track 0.00 -> 4.29 mm
- net S$33: track 0.00 -> 4.29 mm
- net S$32: track 0.00 -> 4.29 mm
- net S$31: track 0.00 -> 4.29 mm
- net S$30: track 0.00 -> 4.29 mm
- net S$29: track 0.00 -> 4.29 mm
- net S$28: track 0.00 -> 4.29 mm
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Other:
- board text added: "27.07.20"
- board text removed: "26.07.20"
