File: Platinen/100-Arduino_fuer_LEDs_Mainboard/Arduino_fuer_LEDs_DCC_4.brd (EAGLE design)
At the start: 82.2 x 73.3 mm, 97 parts, among them IC1 7805, IC2 LM393N, J1 Tag/Nacht, U1 WS2812_MODUL, U2 LED NANO, U3 DCC NANO, U4 WS2812_MODUL, X1 RJ10, X2 AK500/2+M, X3 MAB 5SH Conrad: 738247 - VQ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

Commit message: V.:1.5
Parts:
- added COPY_LED: (no value), adafruit:1X03-CLEANBIG
- added H5, H6: MOUNT-HOLE3.0, holes:3,0
- added INP, O1, O2, O3, O4: (no value), con-harting-ml:ML6
Connections:
- new net N$52: INP.4, O3.4, O4.2
- new net N$53: O4.4
- new net N$55: COPY_LED.2, O2.2
- new net N$57: COPY_LED.3, INP.2, O1.2
- new net N$58: O2.4, O3.2
- new net N$60: COPY_LED.1, O1.4
- new net POWER2: INP.6, O1.6, O2.6, O3.6, O4.6
- new net V_5V: INP.1, O1.1, O2.1, O3.1, O4.1
- new net V_GND: INP.3, INP.5, O1.3, O1.5, O2.3, O2.5, O3.3, O3.5, O4.3, O4.5
Routing:
- net N$52: track 0.00 -> 79.8 mm
- net POWER2: track 0.00 -> 75.1 mm
- net V_GND: track 0.00 -> 57.2 mm
- net V_5V: track 0.00 -> 51.8 mm
- net N$57: track 0.00 -> 29.9 mm
- net N$55: track 0.00 -> 12.7 mm
- net N$60: track 0.00 -> 11.6 mm
- net N$58: track 0.00 -> 10.6 mm
- added copper zone on layer 1, net V_5V
- added copper zone on layer 16, net V_GND
Other:
- board size 82.2 x 73.3 mm -> 100 x 73.3 mm
- board text added: "02.08.20"
- board text added: "Normal"
