File: Platinen/100-Arduino_fuer_LEDs_Mainboard/Arduino_fuer_LEDs_DCC_4.sch (EAGLE design)
At the start: 97 parts, among them IC1 7805, IC2 LM393N, J1 Tag/Nacht, U1 WS2812_MODUL, U2 LED NANO, U3 DCC NANO, U4 WS2812_MODUL, X1 RJ10, X2 AK500/2+M, X3 MAB 5SH Conrad: 738247 - VQ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

Commit message: V.:1.5
Parts:
- added COPY_LED: (no value), adafruit:PINHD-1X3CB
- added H5, H6: MOUNT-HOLE3.0, holes:MOUNT-HOLE3.0
- added INP, O1, O2, O3, O4: (no value), con-harting-ml:ML6
Connections:
- new net N$52: INP.4, O3.4, O4.2
- new net N$53: O4.4
- new net N$55: COPY_LED.2, O2.2
- new net N$57: COPY_LED.3, INP.2, O1.2
- new net N$58: O2.4, O3.2
- new net N$60: COPY_LED.1, O1.4
- new net POWER2: INP.6, O1.6, O2.6, O3.6, O4.6
- new net V_5V: INP.1, O1.1, O2.1, O3.1, O4.1
- new net V_GND: INP.3, INP.5, O1.3, O1.5, O2.3, O2.5, O3.3, O3.5, O4.3, O4.5
Other:
- note added: "4-pol or 6-pol connector could be used"
- note added: "LED Platinen und mini Verteiler mit Duplikate Funktion."
- note added: "Wenn Jumper "COPY_LED" die Pins 2 und 3 verbindet, dann bekommt O1 und O2 das gleiche Signal. Das ist zum Testen von speziellen Schaltungen wie der Servo Platine hilfreich. Normalerweise ist 1 und 2 verbunden."
- moved on the sheet: C10, C11, C12, C13, C14, C15, C16, C17, C18, C19, CON1, CON10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
