File: Platinen/100-Arduino_fuer_LEDs_Mainboard/Arduino_fuer_LEDs_DCC_1.8.1.sch (EAGLE design)
At the start: 122 parts, among them CON5 M04B4B-ZR4P, IC1 7805, IC2 LM393N, IC3 74125N, IC4 MCP2515-I/P, IC5 ISO1050, IC6 B0505S-1W, J1 day /night, J2 LocoNet, Q1 BC547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

Commit message: Mainboard Final Version 1.8.1
Parts:
- removed C10, C12: 100nF, rcl:C-EU025-025X050
- removed C11, C13: 100nF, rcl:C-EUC1206
- removed CON1, CON2, CON3, CON4, COPY_LED: (no value), adafruit:PINHD-1X3CB
- removed LED2, LED3: WS2812B5050, adafruit:WS2812B5050
- removed LED4, LED5: WS2812B3535, adafruit:WS2812B3535
- removed SJ4: SOLDERJUMPERNO, SparkFun-Retired:SOLDERJUMPERNO
- removed SJ_NORM: SOLDERJUMPERTRACE, SparkFun-Retired:SOLDERJUMPERTRACE
- added H7: MOUNT-HOLE3.0, holes:MOUNT-HOLE3.0
- added J3, KEY_A7: SOLDERJUMPERNO, SparkFun-Retired:SOLDERJUMPERNO
- added R15: (100), Arduino_fuer_LEDs_DCC_2:R0204/7
- added X7, X9: AK500/2+M, Arduino_fuer_LEDs_DCC_2:AK500/2+M
- C3: VOLTAGE (none) -> 6.3V
- C4: VOLTAGE (none) -> 20V
- MINI_VERT: value SOLDERJUMPERTRACE -> SOLDERJUMPERNO; device SparkFun-Retired:SOLDERJUMPERTRACE -> SparkFun-Retired:SOLDERJUMPERNO
- R9: device rcl:R-EU_0204/5 -> rcl:R-EU_0204/7
Connections:
- removed net N$10: CON4.2, LED3.DO, LED5.DO
- removed net N$11: COPY_LED.1, O1.4, SJ_NORM.2
- removed net N$23: C7.1, KEYBRD_1.8, R14.1, SJ4.2
- net +5V: now also J3.1, X9G$2.KL; no longer C10.1, C11.1, C12.1, C13.1, CON1.1, CON2.1, CON3.1, CON4.1, LED2.VDD, LED3.VDD, LED4.VDD, LED5.VDD
- net A7: now also KEY_A7.1
- net D6: no longer CON1.2, LED2.DI, LED4.DI
- net DT0: no longer CON2.2, LED2.DO, LED4.DO
- net GND: now also KEYBRD_1.2, X7G$1.KL, X7G$3.KL, X9G$1.KL, X9G$3.KL; no longer C10.2, C11.2, C12.2, C13.2, CON1.3, CON2.3, CON3.3, CON4.3, LED2.GND, LED3.GND, LED4.GND, LED5.GND
- net MV_IN: no longer COPY_LED.3
- net MV_OUT: no longer CON3.2, LED3.DI, LED5.DI
- net N$24: now also R15.2
- net N$25: now also KEY_A7.2
- net N$27: now also C7.1, KEYBRD_1.8, R14.1; no longer SJ4.1
- net N$35: now also O1.4; no longer COPY_LED.2, SJ_NORM.1
- net POWER2: now also J3.2, X7G$2.KL
- net SCL: now also R15.1
Other:
- note added: "24.11.22: => Ver. 1.8.1 - Removed JP4 25.11.22: - Additional connections for KEYBRD_1 for analog buttons. (1:A5, 2:GND, 5:A7)"
- note added: "Close if Pin 6 is used for 5V Leave open if it's used for 12V"
- note added: "Jumper verbinden, wenn der Mini-Verteiler abgesägt wird."
- note added: "Only equip when the mini distributor is cut off."
- note added: "Selectrix (Loconet) Mini Verteiler"
- note added: "Ver.: 1.8.1"
- note removed: "Entweder den bedrahteten oder den SMD Kondensator bestücken."
- note removed: "Jumper unterbrechen, wenn der Mini-Verteiler nicht abgesägt wird und an der Hauptplatine bleibt. Der INP Anschluss am Mini-Verteiler wird dann nicht bestückt."
- note removed: "LED Platinen und mini Verteiler mit Duplikate Funktion."
- note removed: "Optional 3535"
- note removed: "Ver.: 1.8"
- note removed: "Wenn Jumper "COPY_LED" die Pins 2 und 3 verbindet, dann bekommt O1 und O2 das gleiche Signal. Das ist zum Testen von speziellen Schaltungen wie der Servo Platine hilfreich. Normalerweise ist 1 und 2 verbunden."
- moved on the sheet: A1, A2, A3, A4, A5, A6, A7, A8, INP, O1, O2, O3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
