File: Platinen/100-Arduino_fuer_LEDs_Mainboard/Arduino_fuer_LEDs_DCC_1.8.2.brd (EAGLE design)
At the start: 100 x 80 mm, 115 parts, among them CON5 M04B4B-ZR4P, IC1 7805, IC2 LM393N, IC3 74125N, IC4 MCP2515-I/P, IC5 ISO1050, IC6 B0505S-1W, J1 day /night, J2 LocoNet, J3 SOLDERJUMPERNO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

Commit message: Update Arduino_fuer_LEDs_DCC_1.8.2.brd
Connections:
- removed net D38_2: R31.2, SJ_LN2.2, U3.D3, U3.D8
- removed net D47_2: IC2.1, R22.1, R30.2, SJ_SX1.2, U3.D4, U3.D7
- new net D37_2: R31.2, SJ_LN2.2, U3.D3, U3.D7
- new net D48_2: IC2.1, R22.1, R30.2, SJ_SX1.2, U3.D4, U3.D8
Routing:
- net D38_2: track 35.8 -> 0.00 mm
- net D48_2: track 0.00 -> 34.4 mm
- net D47_2: track 31.2 -> 0.00 mm
- net D37_2: track 0.00 -> 30.3 mm
- net N$27: track 88.6 -> 87.3 mm

Commit message: Update Arduino_fuer_LEDs_DCC_1.8.2.brd
Parts:
- added R19: 10K, rcl:0207/2V
Connections:
- new net N$11: IC3.10, IC3.13, R19.2, U3.D9
- net +5V: now also R19.1
- net D13: now also IC3.11
- net GND: no longer IC3.10, IC3.12, IC3.13, IC3.9
- net N$15: now also IC3.8
- net N$20: now also IC3.12
- net N$28: now also IC3.9
Routing:
- net N$20: track 15.8 -> 96.5 mm, vias 0 -> 2
- net N$11: track 0.00 -> 76.7 mm, vias 0 -> 2
- net N$28: track 34.1 -> 104.3 mm, vias 0 -> 2
- net N$15: track 29.2 -> 97.5 mm, vias 0 -> 3
- net D13: track 88.7 -> 103.4 mm, vias 3 -> 4
- net MV_OUT: track 196.0 -> 209.6 mm
- net GND: track 673.3 -> 663.1 mm
- net D7: track 89.0 -> 94.5 mm
- net D12: track 113.4 -> 117.4 mm
- net N$3: track 48.6 -> 52.3 mm
- net +5V: track 440.3 -> 443.4 mm
- net N$6: track 14.9 -> 17.0 mm
- net DT0: track 34.9 -> 33.1 mm
- net N$27: track 87.3 -> 88.5 mm
- net MV_IN: track 204.5 -> 203.6 mm
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