File: Platinen/ISO_CAN_Modul/ISO_CAN_Modul.sch (EAGLE design)
At the start: 26 parts, among them CON8 Term, IC1 MCP2515-I/P, IC2 ISO1050, IC3 B0505S-1W, X1 8 MHz, X2 Male, X3 Male, X4 Male, X5 AK500/2+M

Commit message: Logo & R1
Connections:
- net CAN_H: now also R1.2
- net GND2: no longer R1.2
Other:
- note added: "R1 wird auf der Platinenunterseite platziert wenn der stehende Sub-9 verwendet wird."
- note added: "Senkrecht montierter Stecker (Mit etwas Abstand wenn IC-Fassung für IC1 verwendet wird) Vermutlich kann man das IC trotzdem nicht mehr wechseln ;-("
- note removed: "Senkrecht montierter Stecker (Mit etwas Abstand wenn IC-Fassung für IC1 verwendet wird)"
- moved on the sheet: CON8, R1
Changed lines of the file:
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@@
 Falls man mal 3 Platinen stapelm will, dann muss INT
 getrennt werden und CS3 verbunden werden.</text>
-<text x="162.56" y="55.88" size="1.778" layer="97">Senkrecht montierter Stecker
+<text x="162.56" y="63.5" size="1.778" layer="97" align="top-left">Senkrecht montierter Stecker
 (Mit etwas Abstand wenn IC-Fassung
-für IC1 verwendet wird)</text>
+für IC1 verwendet wird)
+Vermutlich kann man das IC trotzdem
+nicht mehr wechseln ;-(</text>
 <text x="182.88" y="124.46" size="1.778" layer="97">Am Platinenrand montierte Stecker.
 Dazu wird die Platine zwischen die Pins
@@
 gerade gebogen werden.
 Nicht in eine Präzisionsfassung.</text>
+<text x="220.98" y="63.5" size="1.778" layer="97">R1 wird auf der
+Platinenunterseite
+platziert wenn der
+stehende Sub-9
+verwendet wird. </text>
 </plain>
 <instances>
@@
 <attribute name="NAME" x="52.578" y="112.776" size="1.778" layer="95" rot="MR180"/>
 </instance>
-<instance part="R1" gate="G$1" x="205.74" y="81.28" smashed="yes" rot="R90">
-<attribute name="NAME" x="204.2414" y="77.47" size="1.778" layer="95" rot="R90"/>
-<attribute name="VALUE" x="204.216" y="81.28" size="1.778" layer="96" rot="R90"/>
-</instance>
-<instance part="CON8" gate="G$1" x="205.74" y="66.04" smashed="yes" rot="MR90">
-<attribute name="VALUE" x="200.66" y="63.5" size="1.778" layer="96" rot="MR90"/>
-<attribute name="NAME" x="211.582" y="63.5" size="1.778" layer="95" rot="MR90"/>
+<instance part="R1" gate="G$1" x="210.82" y="81.28" smashed="yes" rot="R90">
+<attribute name="NAME" x="209.3214" y="77.47" size="1.778" layer="95" rot="R90"/>
+<attribute name="VALUE" x="209.296" y="81.28" size="1.778" layer="96" rot="R90"/>
+</instance>
+<instance part="CON8" gate="G$1" x="210.82" y="66.04" smashed="yes" rot="MR90">
+<attribute name="VALUE" x="205.74" y="63.5" size="1.778" layer="96" rot="MR90"/>
+<attribute name="NAME" x="216.662" y="63.5" size="1.778" layer="95" rot="MR90"/>
 </instance>
 <instance part="LED1" gate="G$1" x="157.48" y="83.82" smashed="yes">
@@
 <wire x1="180.34" y1="93.98" x2="185.42" y2="93.98" width="0.1524" layer="91"/>
 <wire x1="185.42" y1="93.98" x2="208.28" y2="93.98" width="0.1524" layer="91"/>
-<wire x1="208.28" y1="93.98" x2="223.52" y2="93.98" width="0.1524" layer="91"/>
+<wire x1="208.28" y1="93.98" x2="213.36" y2="93.98" width="0.1524" layer="91"/>
+<wire x1="213.36" y1="93.98" x2="223.52" y2="93.98" width="0.1524" layer="91"/>
 <wire x1="223.52" y1="93.98" x2="231.14" y2="93.98" width="0.1524" layer="91"/>
 <wire x1="231.14" y1="93.98" x2="233.68" y2="96.52" width="0.1524" layer="91"/>
@@
 <junction x="208.28" y="93.98"/>
 <pinref part="CON8" gate="G$1" pin="2"/>
-<wire x1="208.28" y1="93.98" x2="208.28" y2="73.66" width="0.1524" layer="91"/>
 <pinref part="X5" gate="G$3" pin="KL"/>
 <wire x1="236.22" y1="116.84" x2="223.52" y2="116.84" width="0.1524" layer="91"/>
@@
 <junction x="223.52" y="116.84"/>
 <label x="226.06" y="121.92" size="1.778" layer="95"/>
+<wire x1="213.36" y1="73.66" x2="213.36" y2="93.98" width="0.1524" layer="91"/>
+<junction x="213.36" y="93.98"/>
 </segment>
 </net>
@@
 <label x="167.64" y="96.52" size="1.778" layer="95"/>
 <pinref part="X2" gate="-1" pin="7"/>
-<wire x1="226.06" y1="96.52" x2="195.58" y2="96.52" width="0.1524" layer="91"/>
+<wire x1="226.06" y1="96.52" x2="210.82" y2="96.52" width="0.1524" layer="91"/>
+<wire x1="210.82" y1="96.52" x2="195.58" y2="96.52" width="0.1524" layer="91"/>
 <wire x1="195.58" y1="96.52" x2="153.67" y2="96.52" width="0.1524" layer="91"/>
 <wire x1="180.34" y1="68.58" x2="180.34" y2="66.04" width="0.1524" layer="91"/>
@@
 <junction x="226.06" y="96.52"/>
 <label x="226.06" y="111.76" size="1.778" layer="95"/>
+<pinref part="R1" gate="G$1" pin="2"/>
+<wire x1="210.82" y1="86.36" x2="210.82" y2="96.52" width="0.1524" layer="91"/>
+<junction x="210.82" y="96.52"/>
 </segment>
 </net>
@@
 <wire x1="218.44" y1="91.44" x2="218.44" y2="86.36" width="0.1524" layer="91"/>
 <junction x="218.44" y="91.44"/>
-<pinref part="R1" gate="G$1" pin="2"/>
-<wire x1="205.74" y1="86.36" x2="205.74" y2="91.44" width="0.1524" layer="91"/>
 <wire x1="157.48" y1="68.58" x2="170.18" y2="68.58" width="0.1524" layer="91"/>
 <junction x="170.18" y="68.58"/>
@@
 <pinref part="CON8" gate="G$1" pin="1"/>
 <pinref part="R1" gate="G$1" pin="1"/>
-<wire x1="205.74" y1="73.66" x2="205.74" y2="76.2" width="0.1524" layer="91"/>
-</segment>
-</net>
+<wire x1="210.82" y1="73.66" x2="210.82" y2="76.2" width="0.1524" layer="91"/>
+</segment>
+</net>

Commit message: Schaltplan - Netznamen ergänzt - Tippfehler korrigiert
Board
- SilkTop: Datum in sichtbaren Bereich verschoben
- Beschriftungen
	X5 verkleinert & verschoben, 
	IC1/MCP verschoben
	GREEN wie Red/Blue ausgerichtet
	Led1-3 ausgerichtet
	eine Beschriftung 'Male' weg (unter X5)
        und diverse andere Überlappungen behoben
	
- nachdem man X3 und X4 nicht falsch einbauen kann habe ich die Pin Beschriftungen 1 & 5 entfernt 
- Bauteilnamen R1-R3 passend zu Led1-Led3, Name von Led1 und Led3 vertauscht, ist am Board schöner
- Trennlinie auf der Oberseite entfernt, weil auch unten vorhanden. Damit ist mehr Platz für den Board Text
- Leiterbahnen verschoben für bessere RatsNest Abdeckung, zwei neue Durchkontaktierungen
Parts:
- removed R11: 2K2, resistor:R-EU_R0805
- removed R12: 1K, resistor:R-EU_M0805
- added R3: 1K, resistor:R-EU_M0805
- added R4: 120, resistor:R-EU_0204/7
- LED1: value Green -> Red
- LED3: value Red -> Green
- R1: value 120 -> 1K; device resistor:R-EU_0204/7 -> resistor:R-EU_M0805
- R2: value 1K -> 2K2
Connections:
- net N$1 renamed TXCAN
- net N$10 renamed CS_INT
- net N$11 renamed VCC2_EXT
- net N$2 renamed RXCAN
- net N$3 renamed OSC2
- net N$4 renamed OSC1
- net N$6 renamed CS_J1
- net N$8 renamed CS
- removed net N$12: CON8.1, R1.1
- removed net N$14: LED3.C, R12.1
- removed net N$5: LED1.C, R2.2
- removed net N$7: LED2.C, R11.1
- new net LED1: LED1.C, R1.1
- new net LED2: LED2.C, R2.1
- new net LED3: LED3.C, R3.2
- new net TERM: CON8.1, R4.1
- net +5V: now also LED1.A; no longer LED3.A
- net CAN_H: now also R4.2; no longer R1.2
- net GND2: now also R3.1; no longer R2.1
- net N$30: now also R1.2; no longer R12.2
- net N$9: now also R2.2; no longer R11.2
- net VCC2: now also LED3.A; no longer LED1.A
Other:
- note added: "Die rechte Seite des CAN Transceivers (VCC2) kann entweder vom Empfänger mit 5V gespeist werden über einen DC/DC Wandler."
- note added: "Mit dem Lötjumper CS1 und CS2 können zwei Platinen übereinander montiert werden. Bei der einen Platine wird der Chip Select über CS1 gemacht, bei der anderen über CS2. CS1 muss dazu getrennt werden. Falls man mal 3 Platinen stapeln will, dann muss INT getrennt werden und CS3 verbunden werden."
- note removed: "Die Rechte Seite des CAN Transceivers (VCC2) kann entweder vom Empfänger mit 5V gespeist werden über einen DC/DC Wandler."
- note removed: "Mit dem Lötjumper CS1 und CS2 können zwei Platinen übereinander montiert werden. Bei der einen Platine wird der Chip Select über CS1 gemacht, bei der anderen über CS2. CS1 muss dazu getrennt werden. Falls man mal 3 Platinen stapelm will, dann muss INT getrennt werden und CS3 verbunden werden."
- moved on the sheet: LED1, LED3, R1, R2
Changed lines of the file:
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@@
 <?xml version="1.0" encoding="utf-8"?>
 <!DOCTYPE eagle SYSTEM "eagle.dtd">
-<eagle version="9.5.2">
+<eagle version="9.6.2">
 <drawing>
 <settings>
@@
 <part name="C3" library="capacitor-wima" deviceset="C" device="2.5/2" value="100 nF"/>
 <part name="LED2" library="led" deviceset="LED" device="CHIPLED_0805" package3d_urn="urn:adsk.eagle:package:15821/1" value="Blue"/>
-<part name="R11" library="resistor" deviceset="R-EU_" device="R0805" value="2K2"/>
+<part name="R2" library="resistor" deviceset="R-EU_" device="M0805" value="2K2"/>
 <part name="SUPPLY61" library="supply2" deviceset="+5V" device=""/>
-<part name="LED3" library="led" deviceset="LED" device="CHIPLED_0805" package3d_urn="urn:adsk.eagle:package:15821/1" value="Red"/>
-<part name="R12" library="resistor" deviceset="R-EU_" device="M0805" value="1K"/>
+<part name="LED1" library="led" deviceset="LED" device="CHIPLED_0805" package3d_urn="urn:adsk.eagle:package:15821/1" value="Red"/>
+<part name="R1" library="resistor" deviceset="R-EU_" device="M0805" value="1K"/>
 <part name="CAN1" library="ISO_CAN_Modul" deviceset="MCP2515_ISO_CAN_PINS" device=""/>
 <part name="SUPPLY7" library="supply2" deviceset="+5V" device=""/>
@@
 <part name="INT" library="SparkFun-Retired" deviceset="SOLDERJUMPER" device="TRACE" value="SOLDERJUMPERTRACE"/>
 <part name="CS3" library="SparkFun-Retired" deviceset="SOLDERJUMPER" device="NO"/>
-<part name="R1" library="resistor" deviceset="R-EU_" device="0204/7" value="120"/>
+<part name="R4" library="resistor" deviceset="R-EU_" device="0204/7" value="120"/>
 <part name="CON8" library="SparkFun-Connectors" deviceset="M02" device="PTH" value="Term"/>
-<part name="LED1" library="led" deviceset="LED" device="CHIPLED_0805" package3d_urn="urn:adsk.eagle:package:15821/1" value="Green"/>
-<part name="R2" library="resistor" deviceset="R-EU_" device="M0805" value="1K"/>
+<part name="LED3" library="led" deviceset="LED" device="CHIPLED_0805" package3d_urn="urn:adsk.eagle:package:15821/1" value="Green"/>
+<part name="R3" library="resistor" deviceset="R-EU_" device="M0805" value="1K"/>
 <part name="X5" library="Arduino_fuer_LEDs_DCC_2" deviceset="AK500/2+M" device=""/>
 </parts>
@@
 wird der Chip Select über CS1 gemacht, bei der anderen
 über CS2. CS1 muss dazu getrennt werden.
-Falls man mal 3 Platinen stapelm will, dann muss INT
+Falls man mal 3 Platinen stapeln will, dann muss INT
 getrennt werden und CS3 verbunden werden.</text>
 <text x="162.56" y="63.5" size="1.778" layer="97" align="top-left">Senkrecht montierter Stecker
@@
 <text x="76.2" y="58.42" size="1.778" layer="97" rot="R180">Die LEDs sind optional. Sie leuchten nur,
 wenn das von der Software unterstützt wird.</text>
-<text x="160.02" y="147.32" size="1.778" layer="97" rot="R180">Die Rechte Seite des CAN Transceivers (VCC2)
+<text x="160.02" y="147.32" size="1.778" layer="97" rot="R180">Die rechte Seite des CAN Transceivers (VCC2)
 kann entweder vom Empfänger mit 5V gespeist
 werden  über einen DC/DC Wandler.</text>
@@
 <attribute name="VALUE" x="46.99" y="80.391" size="1.778" layer="96" rot="R180"/>
 </instance>
-<instance part="R11" gate="G$1" x="58.42" y="76.2" smashed="yes">
+<instance part="R2" gate="G$1" x="58.42" y="76.2" smashed="yes">
 <attribute name="NAME" x="54.61" y="77.6986" size="1.778" layer="95"/>
 <attribute name="VALUE" x="54.61" y="72.898" size="1.778" layer="96"/>
@@
 <attribute name="VALUE" x="32.385" y="70.485" size="1.778" layer="96" rot="R90"/>
 </instance>
-<instance part="LED3" gate="G$1" x="43.18" y="68.58" smashed="yes" rot="R90">
+<instance part="LED1" gate="G$1" x="43.18" y="68.58" smashed="yes" rot="R90">
 <attribute name="NAME" x="52.959" y="70.866" size="1.778" layer="95" rot="R180"/>
 <attribute name="VALUE" x="47.498" y="64.897" size="1.778" layer="96" rot="R180"/>
 </instance>
-<instance part="R12" gate="G$1" x="58.42" y="68.58" smashed="yes">
+<instance part="R1" gate="G$1" x="58.42" y="68.58" smashed="yes">
 <attribute name="NAME" x="54.61" y="70.0786" size="1.778" layer="95"/>
 <attribute name="VALUE" x="54.61" y="65.278" size="1.778" layer="96"/>
@@
 <attribute name="NAME" x="52.578" y="112.776" size="1.778" layer="95" rot="MR180"/>
 </instance>
-<instance part="R1" gate="G$1" x="210.82" y="81.28" smashed="yes" rot="R90">
+<instance part="R4" gate="G$1" x="210.82" y="81.28" smashed="yes" rot="R90">
 <attribute name="NAME" x="209.3214" y="77.47" size="1.778" layer="95" rot="R90"/>
 <attribute name="VALUE" x="209.296" y="81.28" size="1.778" layer="96" rot="R90"/>
@@
 <attribute name="NAME" x="216.662" y="63.5" size="1.778" layer="95" rot="MR90"/>
 </instance>
-<instance part="LED1" gate="G$1" x="157.48" y="83.82" smashed="yes">
+<instance part="LED3" gate="G$1" x="157.48" y="83.82" smashed="yes">
 <attribute name="NAME" x="153.416" y="79.121" size="1.778" layer="95" rot="R90"/>
 <attribute name="VALUE" x="161.671" y="80.01" size="1.778" layer="96" rot="R90"/>
 </instance>
-<instance part="R2" gate="G$1" x="157.48" y="73.66" smashed="yes" rot="R90">
+<instance part="R3" gate="G$1" x="157.48" y="73.66" smashed="yes" rot="R90">
 <attribute name="NAME" x="155.9814" y="69.85" size="1.778" layer="95" rot="R90"/>
 <attribute name="VALUE" x="160.782" y="69.85" size="1.778" layer="96" rot="R90"/>
@@
 </busses>
 <nets>
-<net name="N$1" class="0">
+<net name="TXCAN" class="0">
 <segment>
 <pinref part="IC1" gate="G$1" pin="TXCAN"/>
@@
 </segment>
 </net>
-<net name="N$2" class="0">
+<net name="RXCAN" class="0">
 <segment>
 <pinref part="IC2" gate="G$1" pin="RXD"/>
@@
 <pinref part="LED2" gate="G$1" pin="A"/>
 <wire x1="40.64" y1="76.2" x2="38.1" y2="76.2" width="0.1524" layer="91"/>
-<pinref part="LED3" gate="G$1" pin="A"/>
+<pinref part="LED1" gate="G$1" pin="A"/>
 <wire x1="40.64" y1="68.58" x2="38.1" y2="68.58" width="0.1524" layer="91"/>
 <wire x1="38.1" y1="68.58" x2="38.1" y2="72.39" width="0.1524" layer="91"/>
@@
 </segment>
 </net>
-<net name="N$3" class="0">
+<net name="OSC2" class="0">
 <segment>
 <pinref part="IC1" gate="G$1" pin="OSC2"/>
@@
 </segment>
 </net>
-<net name="N$4" class="0">
+<net name="OSC1" class="0">
 <segment>
 <pinref part="IC1" gate="G$1" pin="OSC1"/>
@@
 </segment>
 </net>
-<net name="N$11" class="0">
+<net name="VCC2_EXT" class="0">
 <segment>
 <pinref part="X3" gate="-1" pin="1"/>
@@
 <junction x="226.06" y="96.52"/>
 <label x="226.06" y="111.76" size="1.778" layer="95"/>
-<pinref part="R1" gate="G$1" pin="2"/>
+<pinref part="R4" gate="G$1" pin="2"/>
 <wire x1="210.82" y1="86.36" x2="210.82" y2="96.52" width="0.1524" layer="91"/>
 <junction x="210.82" y="96.52"/>
@@
 <segment>
 <pinref part="IC1" gate="G$1" pin="RX0BF"/>
-<pinref part="R11" gate="G$1" pin="2"/>
+<pinref part="R2" gate="G$1" pin="2"/>
 <wire x1="63.5" y1="76.2" x2="63.5" y2="81.28" width="0.1524" layer="91"/>
 <wire x1="63.5" y1="81.28" x2="71.12" y2="81.28" width="0.1524" layer="91"/>
@@
 <wire x1="68.58" y1="78.74" x2="71.12" y2="78.74" width="0.1524" layer="91"/>
 <wire x1="68.58" y1="68.58" x2="68.58" y2="78.74" width="0.1524" layer="91"/>
-<pinref part="R12" gate="G$1" pin="2"/>
+<pinref part="R1" gate="G$1" pin="2"/>
 <wire x1="63.5" y1="68.58" x2="68.58" y2="68.58" width="0.1524" layer="91"/>
 </segment>
@@
 <junction x="157.48" y="99.06"/>
 <label x="160.02" y="106.68" size="1.778" layer="95" rot="R90"/>
-<pinref part="LED1" gate="G$1" pin="A"/>
+<pinref part="LED3" gate="G$1" pin="A"/>
 <wire x1="157.48" y1="99.06" x2="157.48" y2="86.36" width="0.1524" layer="91"/>
 </segment>
 </net>
-<net name="N$6" class="0">
+<net name="CS_J1" class="0">
 <segment>
 <pinref part="J1" gate="G$1" pin="1"/>
@@
 </segment>
 </net>
-<net name="N$8" class="0">
+<net name="CS" class="0">
 <segment>
 <pinref part="CS1" gate="1" pin="2"/>
@@
 <wire x1="157.48" y1="68.58" x2="170.18" y2="68.58" width="0.1524" layer="91"/>
 <junction x="170.18" y="68.58"/>
-<pinref part="R2" gate="G$1" pin="1"/>
+<pinref part="R3" gate="G$1" pin="1"/>
 <label x="162.56" y="68.58" size="1.778" layer="95"/>
 </segment>
 </net>
-<net name="N$10" class="0">
+<net name="CS_INT" class="0">
 <segment>
 <pinref part="CAN1" gate="G$1" pin="INT"/>
@@
 </segment>
 </net>
-<net name="N$7" class="0">
+<net name="LED2" class="0">
 <segment>
 <pinref part="LED2" gate="G$1" pin="C"/>
-<pinref part="R11" gate="G$1" pin="1"/>
+<pinref part="R2" gate="G$1" pin="1"/>
 <wire x1="48.26" y1="76.2" x2="53.34" y2="76.2" width="0.1524" layer="91"/>
 </segment>
 </net>
-<net name="N$12" class="0">
+<net name="TERM" class="0">
 <segment>
 <pinref part="CON8" gate="G$1" pin="1"/>
+<pinref part="R4" gate="G$1" pin="1"/>
+<wire x1="210.82" y1="73.66" x2="210.82" y2="76.2" width="0.1524" layer="91"/>
+</segment>
+</net>
+<net name="LED1" class="0">
+<segment>
+<pinref part="LED1" gate="G$1" pin="C"/>
 <pinref part="R1" gate="G$1" pin="1"/>
-<wire x1="210.82" y1="73.66" x2="210.82" y2="76.2" width="0.1524" layer="91"/>
-</segment>
-</net>
-<net name="N$14" class="0">
-<segment>
+<wire x1="48.26" y1="68.58" x2="53.34" y2="68.58" width="0.1524" layer="91"/>
+</segment>
+</net>
+<net name="LED3" class="0">
+<segment>
+<pinref part="R3" gate="G$1" pin="2"/>
 <pinref part="LED3" gate="G$1" pin="C"/>
-<pinref part="R12" gate="G$1" pin="1"/>
-<wire x1="48.26" y1="68.58" x2="53.34" y2="68.58" width="0.1524" layer="91"/>
-</segment>
-</net>
-<net name="N$5" class="0">
-<segment>
-<pinref part="R2" gate="G$1" pin="2"/>
-<pinref part="LED1" gate="G$1" pin="C"/>
-</segment>
-</net>
+</segment>
+</net>
