File: Platinen/620-CAN-Modul-galv-getr/ISO_CAN_Module.sch (EAGLE design)
At the start: 26 parts, among them CON8 Term, IC1 MCP2515-I/P, IC2 ISO1050, IC3 B0505S-1W, X1 8 MHz, X2 Male, X3 Male, X4 Male, X5 AK500/2+M

Commit message: Final Version
Parts:
- added C4: 100 nF, capacitor-wima:C2.5/2
- added J2, J3, J4, J5: (no value), SparkFun-Connectors:M01S
Connections:
- net +5V: now also J4.1
- net GND2: now also C4.1
- net OSC1: now also J3.1
- net OSC2: now also J2.1
- net VCC2: now also C4.2, J5.1
Changed lines of the file:
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@@
 <?xml version="1.0" encoding="utf-8"?>
 <!DOCTYPE eagle SYSTEM "eagle.dtd">
-<eagle version="9.6.2">
+<eagle version="9.5.2">
 <drawing>
 <settings>
@@
 <part name="R3" library="resistor" deviceset="R-EU_" device="M0805" value="1K"/>
 <part name="X5" library="Arduino_fuer_LEDs_DCC_2" deviceset="AK500/2+M" device=""/>
+<part name="J2" library="SparkFun-Connectors" deviceset="M01S" device=""/>
+<part name="J3" library="SparkFun-Connectors" deviceset="M01S" device=""/>
+<part name="J4" library="SparkFun-Connectors" deviceset="M01S" device=""/>
+<part name="C4" library="capacitor-wima" deviceset="C" device="2.5/2" value="100 nF"/>
+<part name="J5" library="SparkFun-Connectors" deviceset="M01S" device=""/>
 </parts>
 <sheets>
@@
 <attribute name="VALUE" x="252.73" y="125.603" size="1.778" layer="96" rot="R180"/>
 </instance>
+<instance part="J2" gate="G$1" x="109.22" y="76.2" smashed="yes" rot="R90"/>
+<instance part="J3" gate="G$1" x="109.22" y="86.36" smashed="yes" rot="R90"/>
+<instance part="J4" gate="G$1" x="109.22" y="101.6" smashed="yes" rot="R90"/>
+<instance part="C4" gate="G$1" x="162.56" y="124.46" smashed="yes" rot="R180">
+<attribute name="NAME" x="166.116" y="124.079" size="1.778" layer="95" rot="R180"/>
+<attribute name="VALUE" x="171.196" y="129.159" size="1.778" layer="96" rot="R180"/>
+</instance>
+<instance part="J5" gate="G$1" x="162.56" y="129.54" smashed="yes" rot="R270"/>
 </instances>
 <busses>
@@
 <wire x1="109.22" y1="101.6" x2="104.14" y2="101.6" width="0.1524" layer="91"/>
 <junction x="104.14" y="101.6"/>
+<pinref part="J4" gate="G$1" pin="1"/>
+<junction x="109.22" y="101.6"/>
 </segment>
 <segment>
@@
 <wire x1="104.14" y1="77.47" x2="104.14" y2="76.2" width="0.1524" layer="91"/>
 <junction x="104.14" y="76.2"/>
+<pinref part="J2" gate="G$1" pin="1"/>
+<junction x="109.22" y="76.2"/>
 </segment>
 </net>
@@
 <wire x1="104.14" y1="85.09" x2="104.14" y2="86.36" width="0.1524" layer="91"/>
 <junction x="104.14" y="86.36"/>
+<pinref part="J3" gate="G$1" pin="1"/>
+<junction x="109.22" y="86.36"/>
 </segment>
 </net>
@@
 <pinref part="LED3" gate="G$1" pin="A"/>
 <wire x1="157.48" y1="99.06" x2="157.48" y2="86.36" width="0.1524" layer="91"/>
+<pinref part="C4" gate="G$1" pin="2"/>
+<wire x1="157.48" y1="129.54" x2="162.56" y2="129.54" width="0.1524" layer="91"/>
+<junction x="157.48" y="129.54"/>
+<pinref part="J5" gate="G$1" pin="1"/>
+<junction x="162.56" y="129.54"/>
 </segment>
 </net>
@@
 <junction x="193.04" y="91.44"/>
 <wire x1="152.4" y1="124.46" x2="154.94" y2="124.46" width="0.1524" layer="91"/>
-<wire x1="154.94" y1="124.46" x2="154.94" y2="91.44" width="0.1524" layer="91"/>
+<wire x1="154.94" y1="124.46" x2="154.94" y2="121.92" width="0.1524" layer="91"/>
 <junction x="154.94" y="91.44"/>
 <pinref part="IC3" gate="G$1" pin="G-OUT"/>
 <pinref part="X4" gate="-1" pin="3"/>
+<wire x1="154.94" y1="121.92" x2="154.94" y2="91.44" width="0.1524" layer="91"/>
 <wire x1="205.74" y1="104.14" x2="205.74" y2="91.44" width="0.1524" layer="91"/>
 <wire x1="205.74" y1="91.44" x2="193.04" y2="91.44" width="0.1524" layer="91"/>
@@
 <pinref part="R3" gate="G$1" pin="1"/>
 <label x="162.56" y="68.58" size="1.778" layer="95"/>
-</segment>
-</net>
+<pinref part="C4" gate="G$1" pin="1"/>
+<junction x="154.94" y="121.92"/>
+<wire x1="154.94" y1="121.92" x2="162.56" y2="121.92" width="0.1524" layer="91"/>
+</segment>
+</net>
