File: Platinen/620-CAN-Modul-galv-getr/ISO_CAN_Module.sch (EAGLE design)
At the start: 31 parts, among them CON8 Term, IC1 MCP2515-I/P, IC2 ISO1050, IC3 B0505S-1W, X1 8 MHz, X2 Male, X3 Male, X4 Male, X5 AK500/2+M

Commit message: Update Schaltplan
~ Schematic Notes R4 (not R1)
Other:
- note added: "R4 wird auf der Platinenunterseite platziert wenn der stehende Sub-9 verwendet wird."
- note removed: "R1 wird auf der Platinenunterseite platziert wenn der stehende Sub-9 verwendet wird."
Changed lines of the file:
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@@
 <?xml version="1.0" encoding="utf-8"?>
 <!DOCTYPE eagle SYSTEM "eagle.dtd">
-<eagle version="9.5.2">
+<eagle version="9.6.2">
 <drawing>
 <settings>
-<setting alwaysvectorfont="no"/>
+<setting alwaysvectorfont="yes"/>
 <setting verticaltext="up"/>
 </settings>
@@
 gerade gebogen werden.
 Nicht in eine Präzisionsfassung.</text>
-<text x="220.98" y="63.5" size="1.778" layer="97">R1 wird auf der
+<text x="220.98" y="63.5" size="1.778" layer="97">R4 wird auf der
 Platinenunterseite
 platziert wenn der
