File: Platinen/110_MLL-ESP32-Adapter/ESP32-Adapter_V101.sch (EAGLE design)
At the start: 90 parts, among them IC1 ISO1050, J1.7 JUMPER-SMT_2_NO_SILK, J2.2 JUMPER-SMT_2_NO_SILK, J2.3 JUMPER-SMT_2_NO_SILK, J2.4 JUMPER-SMT_2_NO_SILK, J2.5 JUMPER-SMT_2_NO_SILK, J2.6 JUMPER-SMT_2_NO_SILK, J2.7 JUMPER-SMT_2_NO_SILK, J3.2 JUMPER-SMT_2_NO_SILK, J3.3 JUMPER-SMT_2_NO_SILK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

Commit message: Updated Board-Files
Changed lines of the file:
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@@
 <attributes>
 <attribute name="AUTOREN" value="Hardi, Jürgen &amp; Dominik"/>
-<attribute name="DATUM" value="2021-04-05"/>
+<attribute name="DATUM" value="2021-04-28"/>
 <attribute name="PROJEKT" value="MLL - ESP32-Adapter "/>
 </attributes>

Commit message: Update ESP32-Adapter_V101.sch
Other:
- note added: "nicht Bestücken"
Changed lines of the file:
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@@
 <?xml version="1.0" encoding="utf-8"?>
 <!DOCTYPE eagle SYSTEM "eagle.dtd">
-<eagle version="9.6.2">
+<eagle version="9.5.2">
 <drawing>
 <settings>
-<setting alwaysvectorfont="yes"/>
+<setting alwaysvectorfont="no"/>
 <setting verticaltext="up"/>
 </settings>
@@
 <text x="354.33" y="15.24" size="1.778" layer="94">&gt;DATUM</text>
 <text x="354.33" y="10.16" size="1.778" layer="94">&gt;AUTOREN</text>
+<wire x1="157.48" y1="144.78" x2="162.56" y2="139.7" width="0.1524" layer="94"/>
+<text x="165.1" y="139.7" size="1.778" layer="94">nicht
+Bestücken</text>
+<text x="294.64" y="58.42" size="1.778" layer="94">nicht
+Bestücken</text>
+<wire x1="287.02" y1="66.04" x2="292.1" y2="60.96" width="0.1524" layer="94"/>
+<wire x1="287.02" y1="60.96" x2="292.1" y2="66.04" width="0.1524" layer="94"/>
+<wire x1="157.48" y1="139.7" x2="162.56" y2="144.78" width="0.1524" layer="94"/>
 </plain>
 <instances>
