File: Platinen/503-WS2811_MultiUse/503-WS2811-Multi_RV100.brd (EAGLE design)
At the start: 71 x 25 mm, 85 parts, among them M1_IN 4XRM254, M1_OUT 4XRM254, M2_IN 4XRM254, M2_OUT 4XRM254, M3_IN 4XRM254, M3_OUT 4XRM254, U1 WS2811, U10 WS2811, U2 WS2811, U3 WS2811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

Commit message: Upload WS2811-MultiUse
+ 503-WS2811_MultiUse - RV100 20220403
- Version V123 with old files
Parts:
- U$2, U$6: value CON-LABEL_MLLRM200 -> CON-LABEL_MLLRM200_3; device MLL-Dominik-Hardi:CON-LABEL_MLLRM200 -> MLL-Dominik-Hardi:CON-LABEL_MLLRM200_3
- moved U$2 19.6 mm to (15.6, 3.56)
- moved U$6 18.0 mm to (34.4, 3.68)
- renumbered M3_IN to IN, M3_OUT to OUT
Other:
- board text added: "IN"
- board text added: "OUT"
- board text removed: "JLCJLCJLCJLC"
