File: Platinen/503-WS2811_MultiUse/503-WS2811-Multi_RV100.sch (EAGLE design)
At the start: 85 parts, among them M1_IN 4XRM254, M1_OUT 4XRM254, M2_IN 4XRM254, M2_OUT 4XRM254, M3_IN 4XRM254, M3_OUT 4XRM254, U1 WS2811, U10 WS2811, U2 WS2811, U3 WS2811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

Commit message: Upload WS2811-MultiUse
+ 503-WS2811_MultiUse - RV100 20220403
- Version V123 with old files
Parts:
- U$2, U$6: value CON-LABEL_MLLRM200 -> CON-LABEL_MLLRM200_3; device MLL-Dominik-Hardi:CON-LABEL_MLLRM200 -> MLL-Dominik-Hardi:CON-LABEL_MLLRM200_3
- renumbered M3_IN to IN, M3_OUT to OUT
Changed lines of the file:
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@@
 <part name="M1_OUT" library="MLL-Dominik-Hardi" deviceset="4XRM254" device=""/>
 <part name="M2_IN" library="MLL-Dominik-Hardi" deviceset="4XRM254" device=""/>
-<part name="M3_IN" library="MLL-Dominik-Hardi" deviceset="4XRM254" device=""/>
+<part name="IN" library="MLL-Dominik-Hardi" deviceset="4XRM254" device=""/>
 <part name="M2_OUT" library="MLL-Dominik-Hardi" deviceset="4XRM254" device=""/>
-<part name="M3_OUT" library="MLL-Dominik-Hardi" deviceset="4XRM254" device=""/>
+<part name="OUT" library="MLL-Dominik-Hardi" deviceset="4XRM254" device=""/>
 <part name="M1_IN" library="MLL-Dominik-Hardi" deviceset="4XRM254" device=""/>
 <part name="TERM3" library="jumper" library_urn="urn:adsk.eagle:library:252" deviceset="SJ" device="" package3d_urn="urn:adsk.eagle:package:15471/1"/>
@@
 <part name="U$20" library="MLL-Dominik-Hardi" deviceset="4XRM200LONG-NOH_DOUBLE" device=""/>
 <part name="LED1" library="SparkFun-LED" library_urn="urn:adsk.eagle:library:529" deviceset="LED" device="3MM" package3d_urn="urn:adsk.eagle:package:39361/1" value="LED 3MM GREEN"/>
-<part name="U$2" library="MLL-Dominik-Hardi" deviceset="CON-LABEL_MLLRM200" device=""/>
 <part name="U$4" library="MLL-Dominik-Hardi" deviceset="CON-LABEL_MLLRM200_2" device="RGB_M" value="CON-LABEL_MLLRM200_2RGB_M"/>
 <part name="U$5" library="MLL-Dominik-Hardi" deviceset="CON-LABEL_MLLRM200_2" device="RGB"/>
@@
 <part name="U$7" library="MLL-Dominik-Hardi" deviceset="4XRM200LONG-NOH_DOUBLE" device=""/>
 <part name="U$9" library="MLL-Dominik-Hardi" deviceset="4XRM200LONG-NOH_DOUBLE" device=""/>
-<part name="U$6" library="MLL-Dominik-Hardi" deviceset="CON-LABEL_MLLRM200" device=""/>
 <part name="SJ2.2" library="MLL-Dominik-Hardi" deviceset="SJ-CON" device=""/>
 <part name="SJ1.2" library="MLL-Dominik-Hardi" deviceset="SJ-CON" device="" value="DO"/>
 <part name="SJ1.1" library="MLL-Dominik-Hardi" deviceset="SJ-CON" device="" value="DO"/>
+<part name="U$2" library="MLL-Dominik-Hardi" deviceset="CON-LABEL_MLLRM200_3" device=""/>
+<part name="U$6" library="MLL-Dominik-Hardi" deviceset="CON-LABEL_MLLRM200_3" device=""/>
 </parts>
 <sheets>
@@
 <instance part="M1_OUT" gate="G$1" x="119.38" y="236.22" smashed="yes" grouprefs="WS2811-G1"/>
 <instance part="M2_IN" gate="G$1" x="140.97" y="236.22" smashed="yes" rot="MR0" grouprefs="WS2811-G2"/>
-<instance part="M3_IN" gate="G$1" x="274.32" y="236.22" smashed="yes" rot="MR0" grouprefs="WS2811-G3"/>
+<instance part="IN" gate="G$1" x="274.32" y="236.22" smashed="yes" rot="MR0" grouprefs="WS2811-G3"/>
 <instance part="M2_OUT" gate="G$1" x="245.11" y="236.22" smashed="yes" grouprefs="WS2811-G2"/>
-<instance part="M3_OUT" gate="G$1" x="381" y="236.22" smashed="yes" grouprefs="WS2811-G3"/>
+<instance part="OUT" gate="G$1" x="381" y="236.22" smashed="yes" grouprefs="WS2811-G3"/>
 <instance part="M1_IN" gate="G$1" x="13.97" y="236.22" smashed="yes" rot="MR0" grouprefs="WS2811-G1"/>
 <instance part="TERM3" gate="1" x="364.49" y="247.65" smashed="yes" grouprefs="WS2811-G3">
@@
 <attribute name="VALUE" x="108.585" y="44.958" size="1.778" layer="96" font="vector" rot="R90" align="top-left"/>
 </instance>
-<instance part="U$2" gate="G$1" x="144.78" y="35.56" smashed="yes"/>
 <instance part="U$4" gate="G$1" x="160.02" y="35.56" smashed="yes"/>
 <instance part="U$5" gate="G$1" x="160.02" y="27.94" smashed="yes"/>
 <instance part="U$1" gate="G$1" x="144.78" y="27.94" smashed="yes"/>
-<instance part="U$3" gate="G$1" x="129.54" y="35.56" smashed="yes"/>
+<instance part="U$3" gate="G$1" x="144.78" y="35.56" smashed="yes"/>
 <instance part="U$8" gate="G$1" x="82.55" y="153.67" smashed="yes" rot="MR270"/>
 <instance part="U$7" gate="G$1" x="74.93" y="102.87" smashed="yes" rot="R270"/>
 <instance part="U$9" gate="G$1" x="74.93" y="195.58" smashed="yes" rot="R270"/>
-<instance part="U$6" gate="G$1" x="129.54" y="27.94" smashed="yes"/>
 <instance part="SJ2.2" gate="G$1" x="129.54" y="255.27" smashed="yes">
 <attribute name="NAME" x="128.27" y="241.3" size="1.27" layer="95"/>
@@
 <attribute name="VALUE" x="10.16" y="88.9" size="0.6096" layer="95"/>
 </instance>
+<instance part="U$2" gate="G$1" x="129.54" y="35.56" smashed="yes"/>
+<instance part="U$6" gate="G$1" x="129.54" y="27.94" smashed="yes"/>
 </instances>
 <busses>
@@
 <pinref part="SJ3.1" gate="G$1" pin="P$2"/>
 <wire x1="257.81" y1="259.08" x2="260.35" y2="259.08" width="0.1524" layer="91"/>
-<pinref part="M3_OUT" gate="G$1" pin="P$1"/>
-<pinref part="M3_IN" gate="G$1" pin="P$1"/>
+<pinref part="OUT" gate="G$1" pin="P$1"/>
+<pinref part="IN" gate="G$1" pin="P$1"/>
 </segment>
 <segment>
@@
 <pinref part="SJ3.3" gate="G$1" pin="P$2"/>
 <wire x1="257.81" y1="251.46" x2="260.35" y2="251.46" width="0.1524" layer="91"/>
-<pinref part="M3_OUT" gate="G$1" pin="P$3"/>
-<pinref part="M3_IN" gate="G$1" pin="P$3"/>
+<pinref part="OUT" gate="G$1" pin="P$3"/>
+<pinref part="IN" gate="G$1" pin="P$3"/>
 </segment>
 <segment>
@@
 <pinref part="SJ3.2" gate="G$1" pin="P$2"/>
 <wire x1="257.81" y1="255.27" x2="260.35" y2="255.27" width="0.1524" layer="91"/>
-<pinref part="M3_IN" gate="G$1" pin="P$2"/>
+<pinref part="IN" gate="G$1" pin="P$2"/>
 </segment>
 </net>
@@
 <wire x1="377.19" y1="45.72" x2="377.19" y2="99.06" width="0.1524" layer="91" grouprefs="WS2811-G3"/>
 <label x="377.19" y="220.98" size="1.778" layer="95" rot="R90" grouprefs="WS2811-G3"/>
-<pinref part="M3_OUT" gate="G$1" pin="P$2"/>
+<pinref part="OUT" gate="G$1" pin="P$2"/>
 <pinref part="TERM3" gate="1" pin="2"/>
 <wire x1="369.57" y1="247.65" x2="377.19" y2="247.65" width="0.1524" layer="91" grouprefs="WS2811-G3"/>
@@
 <junction x="297.18" y="247.65" grouprefs="WS2811-G3"/>
 <wire x1="297.18" y1="236.22" x2="297.18" y2="247.65" width="0.1524" layer="91" grouprefs="WS2811-G3"/>
-<pinref part="M3_IN" gate="G$1" pin="P$4"/>
+<pinref part="IN" gate="G$1" pin="P$4"/>
 <wire x1="276.86" y1="236.22" x2="297.18" y2="236.22" width="0.1524" layer="91" grouprefs="WS2811-G3"/>
 <wire x1="297.18" y1="247.65" x2="356.87" y2="247.65" width="0.1524" layer="91" grouprefs="WS2811-G3"/>
 <pinref part="TERM3" gate="1" pin="1"/>
-<pinref part="M3_OUT" gate="G$1" pin="P$4"/>
+<pinref part="OUT" gate="G$1" pin="P$4"/>
 <wire x1="356.87" y1="247.65" x2="359.41" y2="247.65" width="0.1524" layer="91" grouprefs="WS2811-G3"/>
 <wire x1="378.46" y1="236.22" x2="356.87" y2="236.22" width="0.1524" layer="91" grouprefs="WS2811-G3"/>
