File: Platinen/Testplatinen/210 & 211 - MLL-Range-Extender/211_MLL-Range-Extender-CAT5/211_MLL-Range-Extender-CAT5_v0063.sch (EAGLE design)
At the start: 60 parts, among them IC1D 75176AP, IC1S 75176AD, IC2D 75176AP, IC2S 75176AD, IC3D 75176AP, IC3S 75176AD, IC4D 75176AP, IC4S 75176AD, IC5 WS2812-5050, IC6 WS2812-5050, IC7 WS2812-5050, IC8 WS2812-5050

Commit message: Update - 211_MLL-Range-Extender-CAT5
Parts:
- removed CONR1, CONR2, CONT1, CONT2: PSK_4WS, HD_Kontakte:PSK_4WS
- removed JP1, JP2: (no value), jumper:JP1E
- removed SJ5, SJ6, SJ7, SJ8: (no value), jumper:SJ
- added D1, D2: BAT43, diode:BAT42
- added IC15, IC16, IC17, IC18: WS2812-BB, HD_ICs:WS2812-BB
- added R5, R6, R7, R8: 100R, rcl:R-EU_0207/10
- added SJ1, SJ2: (no value), jumper:SJ
Connections:
- net N$4 renamed LED1-R
- net N$7 renamed LED2_R
- removed net GND1: C1S.1, C1T.1, C2S.1, C2T.1, C5.1, C6.1, CONT1.1, CONT2.1, IC1D.GND, IC1D.R, IC1S.GND, IC1S.R, IC2D.!RE, IC2D.D, IC2D.DE, IC2D.GND, IC2S.!RE, IC2S.D, IC2S.DE, IC2S.GND, IC5.GND, IC6.GND, INPUT.GND, INPUT.GND2, LED1.C, RJ45-SEND.BROWN/WHITE, RJ45-SEND.ORANGE/WHITE
- removed net GND2: C3S.1, C3T.1, C4S.1, C4T.1, C7.1, C8.1, CONR1.1, CONR2.1, CP2.+, IC3D.!RE, IC3D.D, IC3D.DE, IC3D.GND, IC3S.!RE, IC3S.D, IC3S.DE, IC3S.GND, IC4D.GND, IC4D.R, IC4S.GND, IC4S.R, IC7.GND, IC8.GND, LED2.C, OUTPUT.GND, OUTPUT.GND2, RJ45-REC.BROWN/WHITE, RJ45-REC.ORANGE/WHITE
- removed net N$13: IC5.DI, INPUT.DI, SJ5.2
- removed net N$15: IC6.DO, INPUT.DO, SJ6.2
- removed net N$17: IC3D.R, IC3S.R, IC7.DI, SJ7.1
- removed net N$2: INPUT.VCC2, JP1.2
- removed net N$27: IC4D.D, IC4S.D, IC8.DO, SJ8.1
- removed net N$3: IC1D.D, IC1S.D, IC5.DO, SJ5.1
- removed net N$5: IC7.DO, OUTPUT.DI, SJ7.2
- removed net N$6: IC8.DI, OUTPUT.DO, SJ8.2
- removed net N$9: IC2D.R, IC2S.R, IC6.DI, SJ6.1
- removed net VCC1: C1S.2, C1T.2, C2S.2, C2T.2, C5.2, C6.2, CONT1.4, CONT2.4, CP1.+, CP1.-, IC1D.!RE, IC1D.DE, IC1D.VCC, IC1S.!RE, IC1S.DE, IC1S.VCC, IC2D.VCC, IC2S.VCC, IC5.VDD, IC6.VDD, INPUT.VCC, JP1.1, R11.2, RJ45-SEND.BROWN, RJ45-SEND.OPRANGE
- removed net VCC2: C3S.2, C3T.2, C4S.2, C4T.2, C7.2, C8.2, CONR1.4, CONR2.4, CP2.-, IC3D.VCC, IC3S.VCC, IC4D.!RE, IC4D.DE, IC4D.VCC, IC4S.!RE, IC4S.DE, IC4S.VCC, IC7.VDD, IC8.VDD, JP2.1, OUTPUT.VCC, R12.2, RJ45-REC.BROWN, RJ45-REC.OPRANGE
- new net +5V/2: C3S.2, C3T.2, C4S.2, C4T.2, C7.2, C8.2, CP2.+, D2.C, IC17.V, IC17.V1, IC18.V, IC18.V1, IC3D.VCC, IC3S.VCC, IC4D.!RE, IC4D.DE, IC4D.VCC, IC4S.!RE, IC4S.DE, IC4S.VCC, IC7.VDD, IC8.VDD, R12.2, SJ1.1
- new net GND: C1S.1, C1T.1, C2S.1, C2T.1, C5.1, C6.1, CP1.-, IC15.G, IC15.G1, IC16.G, IC16.G1, IC1D.GND, IC1S.GND, IC2D.!RE, IC2D.D, IC2D.DE, IC2D.GND, IC2S.!RE, IC2S.D, IC2S.DE, IC2S.GND, IC5.GND, IC6.GND, INPUT.GND, INPUT.GND2, LED1.C, RJ45-SEND.BLUE, RJ45-SEND.BROWN
- new net GNDA: C3S.1, C3T.1, C4S.1, C4T.1, C7.1, C8.1, CP2.-, IC17.G, IC17.G1, IC18.G, IC18.G1, IC3D.!RE, IC3D.D, IC3D.DE, IC3D.GND, IC3S.!RE, IC3S.D, IC3S.DE, IC3S.GND, IC4D.GND, IC4S.GND, IC7.GND, IC8.GND, LED2.C, OUTPUT.GND, OUTPUT.GND2, RJ45-REC.BLUE, RJ45-REC.BROWN
- new net IC1_R: IC1D.R, IC1S.R
- new net IC4_R: IC4D.R, IC4S.R
- new net R_DI: IC17.DO, IC7.DO, OUTPUT.DI, R7.2
- new net R_DI1: IC17.DI, IC3D.R, IC3S.R, IC7.DI, R7.1
- new net R_DO: IC18.DI, IC8.DI, OUTPUT.DO, R8.2
- new net R_DO_1: IC18.DO, IC4D.D, IC4S.D, IC8.DO, R8.1
- new net T_DI: IC15.DI, IC5.DI, INPUT.DI, R5.2
- new net T_DI-1: IC15.DO, IC1D.D, IC1S.D, IC5.DO, R5.1
- new net T_DO: IC16.DO, IC6.DO, INPUT.DO, R6.2
- new net T_DO-1: IC16.DI, IC2D.R, IC2S.R, IC6.DI, R6.1
- new net VCC: C1S.2, C1T.2, C2S.2, C2T.2, C5.2, C6.2, CP1.+, D1.C, IC15.V, IC15.V1, IC16.V, IC16.V1, IC1D.!RE, IC1D.DE, IC1D.VCC, IC1S.!RE, IC1S.DE, IC1S.VCC, IC2D.VCC, IC2S.VCC, IC5.VDD, IC6.VDD, R11.2, SJ2.1
- new net VCC_T: RJ45-SEND.BLUE/WHITE, RJ45-SEND.BROWN/WHITE, SJ2.2
- new net VDD_IN: D2.A, OUTPUT.VCC
- new net VDD_T: RJ45-REC.BLUE/WHITE, RJ45-REC.BROWN/WHITE, SJ1.2
- net A1: now also RJ45-SEND.ORANGE/WHITE; no longer CONT1.2, RJ45-SEND.BLUE
- net A2: now also RJ45-SEND.GREEN/WHITE; no longer CONT2.3, RJ45-SEND.GREEN
- net A3: now also RJ45-REC.ORANGE/WHITE; no longer CONR1.3, RJ45-REC.BLUE
- net A4: now also RJ45-REC.GREEN/WHITE; no longer CONR2.3, RJ45-REC.GREEN
- net B1: now also RJ45-SEND.OPRANGE; no longer CONT1.3, RJ45-SEND.BLUE/WHITE
- net B2: now also RJ45-SEND.GREEN; no longer CONT2.2, RJ45-SEND.GREEN/WHITE
- net B3: now also RJ45-REC.OPRANGE; no longer CONR1.2, RJ45-REC.BLUE/WHITE
- net B4: now also RJ45-REC.GREEN; no longer CONR2.2, RJ45-REC.GREEN/WHITE
- net N$1: now also D1.A, INPUT.VCC; no longer JP2.2, OUTPUT.VCC2
Other:
- note added: "########## Release Version 1.0.2 ########## Ver0050 & Ver0051 (2022-05-07) ~ Correction connections DI and DO of IC16, IC17 & IC18 ~ Correction CP2 alignment ~ Footprint of IC5 - IC8, as well as IC25-28 exchanged for a clearer imprint of the installation direction ########## Release Version 1.0.1 ########## Ver 0030 (2022-04-18) Release Prototyp Ver 0015 - 0016 (2022-04-16): ~ routing new devices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"
- note removed: "Ver 0015 - 0016 (2022-04-16): ~ routing new devices Ver 0014 (2022-04-16): + LED1, LED2 + R11, R12 + CONT1, CONT2, CONR1, CONR2 Ver 0010 - 0013 (2022-04-16): * first board draft Ver 0001 - 0009 (2022-04-15): * initial planning and elaboration of the basic circuit"
