File: Platinen/550-WS2811_Stepper/Archiv/WS2811_Stepper.brd (EAGLE design)
At the start: 71.4 x 38.7 mm, 50 parts, among them CON1 End SW1, CON2 End SW2, CON3 End SW1H, CON4 STEPPER_CON, CON5 End SW2H, CON6 NEMA17, CON7 LED, IC1 4017N, J10 , M1 BOARD_A4988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

Commit message: Update-Layout-Platine-550
Parts:
- moved CON1 3.59 mm to (5.08, 15.9), turned to 0 degrees
- moved CON2 3.59 mm to (7.62, 13.3), turned to 180 degrees
Connections:
- net M1A renamed N$41
- net M1B renamed N$35
- net M2A renamed N$40
- net M2B renamed N$31
- net VCC2 renamed N$7
- net N$6: now also CON1.1, CON2.2; no longer CON1.2, CON2.1
- net N$8: now also CON2.1; no longer CON1.1
- net N$9: now also CON1.2; no longer CON2.2
Other:
- board text added: "https://wiki.mobaledlib.de/"
- board text removed: "https://wiki.mobaledlib.de/p550"
Changed lines of the file:
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@@
 <?xml version="1.0" encoding="utf-8"?>
 <!DOCTYPE eagle SYSTEM "eagle.dtd">
-<eagle version="9.6.2">
+<eagle version="9.5.2">
 <drawing>
 <settings>
@@
 <setting verticaltext="up"/>
 </settings>
-<grid distance="12.5" unitdist="mil" unit="mil" style="lines" multiple="1" display="yes" altdistance="12.5" altunitdist="mil" altunit="mil"/>
+<grid distance="50" unitdist="mil" unit="mil" style="lines" multiple="1" display="yes" altdistance="12.5" altunitdist="mil" altunit="mil"/>
 <layers>
 <layer number="1" name="Top" color="4" fill="1" visible="yes" active="yes"/>
@@
 <layer number="25" name="tNames" color="7" fill="1" visible="yes" active="yes"/>
 <layer number="26" name="bNames" color="7" fill="1" visible="yes" active="yes"/>
-<layer number="27" name="tValues" color="7" fill="1" visible="yes" active="yes"/>
+<layer number="27" name="tValues" color="7" fill="1" visible="no" active="yes"/>
 <layer number="28" name="bValues" color="7" fill="1" visible="no" active="yes"/>
 <layer number="29" name="tStop" color="7" fill="3" visible="no" active="yes"/>
@@
 <layer number="43" name="vRestrict" color="2" fill="10" visible="no" active="yes"/>
 <layer number="44" name="Drills" color="7" fill="1" visible="no" active="yes"/>
-<layer number="45" name="Holes" color="7" fill="1" visible="no" active="yes"/>
+<layer number="45" name="Holes" color="7" fill="1" visible="yes" active="yes"/>
 <layer number="46" name="Milling" color="3" fill="1" visible="no" active="yes"/>
 <layer number="47" name="Measures" color="7" fill="1" visible="no" active="yes"/>
@@
 <text x="10.795" y="2.8575" size="1.016" layer="25">GND</text>
 <text x="10.4775" y="35.2425" size="1.016" layer="25">GND</text>
-<text x="0.3175" y="13.0175" size="1.016" layer="25">SW1</text>
+<text x="0.3175" y="12.7" size="1.016" layer="25">SW1</text>
 <text x="0.3175" y="6.35" size="1.016" layer="25">SW1</text>
 <text x="0.3175" y="15.24" size="1.016" layer="25">SW2</text>
 <text x="0.3175" y="8.89" size="1.016" layer="25">SW2</text>
-<text x="53.0225" y="1.905" size="1.016" layer="25" rot="R90">Fast</text>
+<text x="53.0225" y="1.27" size="1.016" layer="25" rot="R90">Fast</text>
 <text x="26.3525" y="2.2225" size="1.016" layer="25" rot="R90">Slow</text>
 <text x="0.3175" y="17.4625" size="1.016" layer="25">End Switch NC</text>
 <text x="0.3175" y="10.4775" size="1.016" layer="25">End SW Hall</text>
-<text x="68.8975" y="29.845" size="1.016" layer="25" rot="R90">+12V</text>
-<text x="68.8975" y="34.6075" size="1.016" layer="25" rot="R90">GND</text>
+<text x="67.6275" y="30.7975" size="1.016" layer="25">+12V</text>
+<text x="67.6275" y="34.6075" size="1.016" layer="25">GND</text>
 <text x="6.35" y="4.7625" size="0.8128" layer="25">GND</text>
 <text x="9.525" y="4.7625" size="0.8128" layer="25">IN</text>
 <text x="11.7475" y="13.0175" size="1.016" layer="25" rot="R90">Norm.
 Closed</text>
-<text x="53.34" y="5.08" size="1.27" layer="25">WS2811 Stepper</text>
-<text x="65.7225" y="1.5875" size="1.016" layer="25" rot="R180">by Hardi</text>
+<text x="53.34" y="0.3175" size="1.27" layer="25">WS2811 Stepper</text>
+<text x="70.485" y="6.35" size="1.016" layer="25" rot="R180">by Hardi</text>
 <text x="5.08" y="21.9075" size="1.016" layer="25" rot="R90">GND</text>
 <text x="0.9525" y="24.765" size="1.016" layer="25" rot="R90">+5V</text>
@@
 <text x="16.1925" y="21.2725" size="1.27" layer="26" rot="MR0">WS2811 Stepper</text>
 <text x="6.985" y="17.78" size="1.016" layer="26" rot="MR0">by Hardi</text>
-<text x="62.23" y="8.89" size="1.016" layer="25" rot="R180">&gt;Ver</text>
+<text x="64.135" y="6.35" size="1.016" layer="25" rot="R180">&gt;Ver</text>
 <text x="16.1925" y="19.3675" size="1.016" layer="26" rot="MR0">&gt;Ver</text>
 <text x="26.67" y="1.27" size="1.016" layer="25" rot="R180">&gt;Date</text>
 <text x="16.1925" y="17.4625" size="1.016" layer="26" rot="MR0">&gt;Date</text>
-<text x="53.34" y="11.7475" size="1.016" layer="26" rot="MR0">https://wiki.mobaledlib.de/p550</text>
+<text x="48.895" y="11.43" size="1.016" layer="26" rot="MR0">https://wiki.mobaledlib.de/</text>
 <text x="68.58" y="34.29" size="1.27" layer="16" font="vector" ratio="15" rot="MR0">Bot</text>
 <text x="69.85" y="6.6675" size="1.27" layer="16" font="vector" ratio="15" rot="MR0">by Hardi</text>
-<text x="59.69" y="33.3375" size="1.27" layer="1" font="vector" ratio="15" rot="R90">Top</text>
+<text x="66.04" y="34.29" size="1.27" layer="1" font="vector" ratio="15">Top</text>
 <text x="63.1825" y="6.6675" size="1.27" layer="1" font="vector" ratio="15">by Hardi</text>
 <text x="31.115" y="20.32" size="1.016" layer="26" rot="MR0">Idee von Erich
 und Michael</text>
-<text x="67.6275" y="28.2575" size="1.016" layer="25">+LED</text>
+<text x="67.6275" y="26.9875" size="1.016" layer="25">+LED</text>
 <text x="58.1025" y="16.51" size="0.762" layer="26" rot="MR90">MS3
    -
@@
 </plain>
 <attributes>
-<attribute name="DATE" value="29.05.21"/>
-<attribute name="VER" value="Ver: 1.0.1"/>
+<attribute name="DATE" value="01.05.21"/>
+<attribute name="VER" value="Ver: 1.0"/>
 </attributes>
 <variantdefs>
@@
 <elements>
 <element name="6=12V" library="SparkFun-Retired" package="SJ_2S-NO" value="SOLDERJUMPERNO" x="19.05" y="35.56" smashed="yes" rot="MR0">
-<attribute name="NAME" x="24.7205" y="34.925" size="1.016" layer="26" rot="MR0"/>
+<attribute name="NAME" x="24.403" y="34.925" size="1.016" layer="26" rot="MR0"/>
 </element>
 <element name="6=5V" library="SparkFun-Retired" package="SJ_2S-NO" value="SOLDERJUMPERNO" x="7.62" y="31.75" smashed="yes" rot="MR180">
-<attribute name="NAME" x="9.252" y="32.7025" size="1.016" layer="26" rot="MR180"/>
+<attribute name="NAME" x="8.9345" y="32.7025" size="1.016" layer="26" rot="MR180"/>
 </element>
 <element name="C1" library="resistor" package="C050-024X044" value="220nF" x="33.02" y="20.955" smashed="yes" rot="R90">
@@
 <attribute name="VALUE" x="53.2892" y="24.7142" size="1.016" layer="25" ratio="10" rot="R270"/>
 </element>
-<element name="CON2" library="SparkFun-Connectors" package="1X02" value="End SW2" x="5.08" y="15.875" smashed="yes"/>
-<element name="CON1" library="SparkFun-Connectors" package="1X02" value="End SW1" x="7.62" y="13.335" smashed="yes" rot="R180"/>
+<element name="CON1" library="SparkFun-Connectors" package="1X02" value="End SW1" x="5.08" y="15.875" smashed="yes"/>
+<element name="CON2" library="SparkFun-Connectors" package="1X02" value="End SW2" x="7.62" y="13.335" smashed="yes" rot="R180"/>
 <element name="CON4" library="Connectors_Inline3_7" package="STEPPER_CON" value="STEPPER_CON" x="58.42" y="10.4775" smashed="yes"/>
 <element name="D1" library="diode" package="DO35-7" value="1N4148" x="20.32" y="12.065" smashed="yes" rot="R180">
@@
 </element>
 <element name="TERM" library="SparkFun-Retired" package="SJ_2S-NO" value="SOLDERJUMPERNO" x="4.445" y="33.02" smashed="yes" rot="MR90">
-<attribute name="NAME" x="3.1305" y="32.385" size="0.8128" layer="26" rot="MR0"/>
+<attribute name="NAME" x="3.448" y="32.385" size="0.8128" layer="26" rot="MR0"/>
 </element>
 <element name="U2R" library="S3PO_Modul_WS2811" package="S3PO_MODUL_WS2811_SOUND_MP3-TF-16P_WS2811_AND_ATTINY_WS2811_DIP08" value="WS2811" x="43.18" y="22.225" smashed="yes" rot="R270">
@@
 <attribute name="OC_NEWARK" value="unknown" x="59.69" y="3.175" size="1.778" layer="27" display="off"/>
 <attribute name="POPULARITY" value="41" x="59.69" y="3.175" size="1.778" layer="27" display="off"/>
-<attribute name="VALUE" x="52.705" y="0.381" size="1.016" layer="25" ratio="10"/>
+<attribute name="VALUE" x="52.705" y="4.826" size="1.016" layer="25" ratio="10"/>
 </element>
 <element name="H4" library="holes" package="2,0" value="MOUNT-HOLE2.0" x="55.88" y="36.195" smashed="yes"/>
@@
 <wire x1="20.2692" y1="10.7442" x2="20.2692" y2="17.6784" width="0.2032" layer="16"/>
 </signal>
-<signal name="M2B">
+<signal name="N$31">
 <contactref element="M1" pad="M2AB"/>
 <contactref element="CON4" pad="2"/>
@@
 <wire x1="65.405" y1="17.78" x2="60.96" y2="13.335" width="0.254" layer="1"/>
 </signal>
-<signal name="M2A">
+<signal name="N$40">
 <contactref element="M1" pad="M2A"/>
 <contactref element="CON4" pad="4"/>
@@
 <wire x1="67.945" y1="18.66763125" x2="67.945" y2="17.78" width="0.254" layer="1"/>
 </signal>
-<signal name="M1A">
+<signal name="N$41">
 <contactref element="M1" pad="M1A"/>
 <contactref element="CON4" pad="3"/>
@@
 <wire x1="59.3249375" y1="21.4884" x2="65.88896875" y2="21.4884" width="0.254" layer="1"/>
 </signal>
-<signal name="M1B">
+<signal name="N$35">
 <contactref element="M1" pad="M1B"/>
 <contactref element="CON4" pad="1"/>
@@
 <wire x1="49.05655" y1="32.258" x2="50.00345" y2="32.258" width="0.2032" layer="1"/>
 </signal>
-<signal name="VCC2">
+<signal name="N$7">
 <contactref element="SV1" pad="6"/>
 <contactref element="SV3" pad="6"/>
@@
 </signal>
 <signal name="N$6">
-<contactref element="CON2" pad="1"/>
-<contactref element="CON1" pad="2"/>
+<contactref element="CON1" pad="1"/>
+<contactref element="CON2" pad="2"/>
 <contactref element="M1" pad="ENABLE"/>
 <contactref element="C2" pad="1"/>
@@
 </signal>
 <signal name="N$8">
-<contactref element="CON1" pad="1"/>
+<contactref element="CON2" pad="1"/>
 <contactref element="D1" pad="A"/>
 <contactref element="Q4" pad="S"/>
@@
 </signal>
 <signal name="N$9">
-<contactref element="CON2" pad="2"/>
+<contactref element="CON1" pad="2"/>
 <contactref element="D2" pad="A"/>
 <contactref element="Q3" pad="S"/>
@@
 </signals>
 <mfgpreviewcolors>
-<mfgpreviewcolor name="soldermaskcolor" color="0xC8000000"/>
+<mfgpreviewcolor name="soldermaskcolor" color="0xC8008000"/>
 <mfgpreviewcolor name="silkscreencolor" color="0xFFFEFEFE"/>
 <mfgpreviewcolor name="backgroundcolor" color="0xFF282828"/>
