File: Platinen/550-WS2811_Stepper/Archiv/WS2811_Stepper.sch (EAGLE design)
At the start: 50 parts, among them CON1 End SW1, CON2 End SW2, CON3 End SW1H, CON4 STEPPER_CON, CON5 End SW2H, CON6 NEMA17, CON7 LED, IC1 4017N, J10 , M1 BOARD_A4988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

Commit message: Update-Layout-Platine-550
Connections:
- net M1A renamed N$41
- net M1B renamed N$35
- net M2A renamed N$40
- net M2B renamed N$31
- net VCC2 renamed N$7
- net N$6: now also CON1.1, CON2.2; no longer CON1.2, CON2.1
- net N$8: now also CON2.1; no longer CON1.1
- net N$9: now also CON1.2; no longer CON2.2
Other:
- note added: "Bei einem winzigen Schrittmotor werden keine Endschalter benötigt. Dann entfallen Q1, Q2, D2 & CON1. Stattdessen wird der Jumper NO_END_SW und CON2 verbunden."
- note removed: "Bei einem winzigen Schrittmotor werden keine Endschalter benötigt. Dann entfallen Q1, Q2, D2 & CON2. Stattdessen wird der Jumper NO_END_SW und CON1 verbunden."
- moved on the sheet: CON1, CON2
Changed lines of the file:
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@@
 <?xml version="1.0" encoding="utf-8"?>
 <!DOCTYPE eagle SYSTEM "eagle.dtd">
-<eagle version="9.6.2">
+<eagle version="9.5.2">
 <drawing>
 <settings>
-<setting alwaysvectorfont="yes"/>
+<setting alwaysvectorfont="no"/>
 <setting verticaltext="up"/>
 </settings>
-<grid distance="0.1" unitdist="inch" unit="inch" style="lines" multiple="1" display="no" altdistance="0.01" altunitdist="inch" altunit="inch"/>
+<grid distance="0.1" unitdist="inch" unit="inch" style="lines" multiple="1" display="no" altdistance="0.05" altunitdist="inch" altunit="inch"/>
 <layers>
 <layer number="1" name="Top" color="4" fill="1" visible="no" active="no"/>
@@
 <part name="P+1" library="supply1" library_urn="urn:adsk.eagle:library:371" deviceset="+5V" device=""/>
 <part name="Q2" library="transistor-small-signal" deviceset="BS170" device=""/>
+<part name="CON1" library="SparkFun-Connectors" deviceset="M02" device="PTH" value="End SW1"/>
 <part name="CON2" library="SparkFun-Connectors" deviceset="M02" device="PTH" value="End SW2"/>
-<part name="CON1" library="SparkFun-Connectors" deviceset="M02" device="PTH" value="End SW1"/>
 <part name="D2" library="diode" deviceset="1N4148" device="DO35-7" value="1N4148"/>
 <part name="D1" library="diode" deviceset="1N4148" device="DO35-7" value="1N4148"/>
@@
 <text x="153.67" y="171.45" size="1.778" layer="97" align="top-left">Bei einem winzigen Schrittmotor
 werden keine Endschalter benötigt.
-Dann entfallen Q1, Q2, D2 &amp; CON2.
+Dann entfallen Q1, Q2, D2 &amp; CON1.
 Stattdessen wird der Jumper NO_END_SW
-und CON1 verbunden.</text>
+und CON2 verbunden.</text>
 <text x="224.79" y="57.15" size="1.778" layer="97" align="top-left">Achtung:
 Spannung am A4988 Poti
@@
 <attribute name="VALUE" x="123.19" y="92.71" size="1.778" layer="96" rot="R270"/>
 </instance>
-<instance part="CON2" gate="G$1" x="111.76" y="157.48" smashed="yes" rot="MR270">
+<instance part="CON1" gate="G$1" x="111.76" y="157.48" smashed="yes" rot="MR270">
 <attribute name="VALUE" x="103.886" y="163.83" size="1.778" layer="96" rot="MR270"/>
 <attribute name="NAME" x="105.918" y="160.02" size="1.778" layer="95" rot="MR270"/>
 </instance>
-<instance part="CON1" gate="G$1" x="124.46" y="157.48" smashed="yes" rot="MR270">
+<instance part="CON2" gate="G$1" x="124.46" y="157.48" smashed="yes" rot="MR270">
 <attribute name="VALUE" x="129.286" y="163.322" size="1.778" layer="96" rot="MR270"/>
 <attribute name="NAME" x="118.618" y="160.02" size="1.778" layer="95" rot="MR270"/>
@@
 </segment>
 </net>
-<net name="M2B" class="0">
+<net name="N$31" class="0">
 <segment>
 <pinref part="M1" gate="G$1" pin="2B"/>
@@
 </segment>
 </net>
-<net name="M2A" class="0">
+<net name="N$40" class="0">
 <segment>
 <pinref part="M1" gate="G$1" pin="2A"/>
@@
 </segment>
 </net>
-<net name="M1A" class="0">
+<net name="N$41" class="0">
 <segment>
 <pinref part="M1" gate="G$1" pin="1A"/>
@@
 </segment>
 </net>
-<net name="M1B" class="0">
+<net name="N$35" class="0">
 <segment>
 <wire x1="243.84" y1="96.52" x2="243.84" y2="99.06" width="0.1524" layer="91"/>
@@
 </segment>
 </net>
-<net name="VCC2" class="0">
+<net name="N$7" class="0">
 <segment>
 <pinref part="SV1" gate="1" pin="6"/>
@@
 <net name="N$6" class="0">
 <segment>
-<pinref part="CON2" gate="G$1" pin="1"/>
+<pinref part="CON1" gate="G$1" pin="1"/>
 <wire x1="111.76" y1="149.86" x2="111.76" y2="137.16" width="0.1524" layer="91"/>
-<pinref part="CON1" gate="G$1" pin="2"/>
+<pinref part="CON2" gate="G$1" pin="2"/>
 <wire x1="111.76" y1="137.16" x2="121.92" y2="137.16" width="0.1524" layer="91"/>
 <wire x1="121.92" y1="137.16" x2="121.92" y2="149.86" width="0.1524" layer="91"/>
@@
 <net name="N$8" class="0">
 <segment>
-<pinref part="CON1" gate="G$1" pin="1"/>
+<pinref part="CON2" gate="G$1" pin="1"/>
 <pinref part="D1" gate="G$1" pin="A"/>
 <wire x1="124.46" y1="149.86" x2="124.46" y2="127" width="0.1524" layer="91"/>
@@
 <net name="N$9" class="0">
 <segment>
-<pinref part="CON2" gate="G$1" pin="2"/>
+<pinref part="CON1" gate="G$1" pin="2"/>
 <pinref part="D2" gate="G$1" pin="A"/>
 <wire x1="109.22" y1="149.86" x2="109.22" y2="127" width="0.1524" layer="91"/>
