File: Platinen/100-Arduino_fuer_LEDs_Mainboard/Archiv/V1.8.1/Arduino_fuer_LEDs_DCC_1.8.1.brd (EAGLE design)
At the start: 100 x 80 mm, 113 parts, among them CON5 M04B4B-ZR4P, IC1 7805, IC2 LM393N, IC3 74125N, IC4 MCP2515-I/P, IC5 ISO1050, IC6 B0505S-1W, J1 day /night, J2 LocoNet, J3 SOLDERJUMPERNO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

Commit message: Update LNET
Parts:
- J2: value LocoNet -> LNet
Changed lines of the file:
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@@
 <attribute name="VALUE" x="58.1533" y="47.16145" size="1.27" layer="25" ratio="10" rot="R180"/>
 </element>
-<element name="J2" library="con-tycoelectronics" package="RJ11-NO_SHIELD_NO_MOUNT_HOULE" value="LocoNet" x="97.79" y="30.00375" smashed="yes" rot="R90">
+<element name="J2" library="con-tycoelectronics" package="RJ11-NO_SHIELD_NO_MOUNT_HOULE" value="LNet" x="97.79" y="30.00375" smashed="yes" rot="R90">
 <attribute name="NAME" x="96.67875" y="30.7975" size="1.27" layer="25" rot="R270"/>
 <attribute name="VALUE" x="98.90125" y="29.845" size="1.27" layer="25" ratio="12" rot="R90" align="center"/>
