File: Platinen/100-Arduino_fuer_LEDs_Mainboard/Archiv/V1.8.1/Arduino_fuer_LEDs_DCC_1.8.1.sch (EAGLE design)
At the start: 116 parts, among them CON5 M04B4B-ZR4P, IC1 7805, IC2 LM393N, IC3 74125N, IC4 MCP2515-I/P, IC5 ISO1050, IC6 B0505S-1W, J1 day /night, J2 LocoNet, J3 SOLDERJUMPERNO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

Commit message: Update LNET
Parts:
- removed R19: 10K, rcl:R-EU_0207/2V
- removed SJ_LN2, SJ_SX6: SOLDERJUMPERNO, SparkFun-Retired:SOLDERJUMPERNO
- J2: value LocoNet -> LNet
Connections:
- removed net D37_2: R31.2, SJ_LN2.2, U3.D3, U3.D7
- removed net N$10: IC2B.OUT, SJ_SX6.1
- removed net N$11: IC3C.OE, IC3D.OE, R19.2, U3.D9
- new net D7_2: R31.2, U3.D7
- net +5V: no longer R19.1
- net D13: no longer IC3D.O
- net D2_2: now also IC2B.OUT; no longer SJ_LN2.1, SJ_SX6.2
- net GND: now also IC3C.I, IC3C.OE, IC3D.I, IC3D.OE
- net N$15: no longer IC3C.O
- net N$20: no longer IC3D.I
- net N$28: no longer IC3C.I
Other:
- note added: "24.11.22: => Ver. 1.8.1 - Removed JP4 25.11.22: - Additional connections for KEYBRD_1 for analog buttons. (1:A5, 2:GND, 5:A7)"
- note added: "Bestückung LNet: R21 = NB (Nicht Bestückt) R23 = 10K R24 = 22K R25 = 47K R28 = NB R29 = 150K R30 = 220K R31 = 10K SJ_LN1 = Verb. SJ_SX1 = Offen SJ_SX2 = Offen SJ_SX3 = Offen SJ_SX4 = Verb. SJ_SX5 = Offen Bestückung Selectrix: (Abweichungen zum Schaltplan) R29 = NB R30 = NB R31 = NB J2 = NB Q1 = NB"
- note added: "DCC / SX LNet"
- note added: "LN"
- note added: "Pinbelegung: https://www.digit-electronic.de/ Info/RJ45 Patchkabel SJ_SX4 wird verbunden wenn ein Pfostenstecker anstelle des RJ45 verwendet wird. Außerdem muß er bei LNet verbunden werden."
- note added: "Revision History: 06.03.19: First Version 27.07.19: Corrected Labeling 04.04.20: Added SJ4, C7, R14 (analog Tatser) 03.06.20: Added R26 (Pull Down für TX) 29.07.20: Added Prg_Boot jumper 30.07.20: Added C8, C9, R27 (analog Taster) - Removed LNet - Removed CV read option - Added Selextrix OP and connectors - Added opt power supply terminal - Added 5V step down regulator - CAN connector could be us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"
- note added: "Revision History: 31.08.20: - Corrected the LED PCBs (Ver. 1.5 was totaly wrong) - swaped the Input/Output pins (3-Pin header = Input) - corrected the pin assignement of the 3535 WS2812 18.10.20: - Corrected the output of the last connector 31.10.22: - New size of te LED modules - Additional normaly colosed Solder Jumper 05.11.22: - Moved the Selectrix part to this sheet - Added LNet components"
- note added: "Selectrix (LNet) Mini Verteiler"
- note added: "Selectrix und LNet (Seite 2)"
- note added: "ToDo: - Correct LED0 / LEDn text (PCB)"
- note added: "Ver.: 1.8.1"
- note added: "WS2811/WS2812 LED Ansteuerung DCC, Selectrix, CAN LNet"
- note added: "nu = Not used by LNet"
- note removed: "10K"
- note removed: "22K"
- note removed: "24.11.22: => Ver. 1.8.1 - Removed JP4 25.11.22: - Additional connections for KEYBRD_1 for analog buttons. (1:A5, 2:GND, 5:A7) 19.12.22: => Ver. 1.8.2 - Corrected LED0/n text (PCB) 21.12.22: - Spare 74125 used to replace Prg_Boot Jumpers"
- note removed: "47K"
- note removed: "Bestückung Loconet: R21 = NB (Nicht Bestückt) R23 = 10K R24 = 22K R25 = 47K R28 = NB R29 = 150K R30 = 220K R31 = 10K SJ_LN1 = Verb. SJ_LN2 = Verb. SJ_SX1 = Offen SJ_SX2 = Offen SJ_SX3 = Offen SJ_SX4 = Verb. SJ_SX5 = Offen SJ_SX6 = Offen Bestückung Selectrix: (Abweichungen zum Schaltplan) R29 = NB R30 = NB R31 = NB J2 = NB Q1 = NB"
- note removed: "DCC / SX LocoNet"
- note removed: "LN RX"
- note removed: "LN TX"
- note removed: "NB"
- note removed: "Pinbelegung: https://www.digit-electronic.de/ Info/RJ45 Patchkabel SJ_SX4 wird verbunden wenn ein Pfostenstecker anstelle des RJ45 verwendet wird. Außerdem muß er bei LocoNet verbunden werden."
- note removed: "Revision History: 06.03.19: First Version 27.07.19: Corrected Labeling 04.04.20: Added SJ4, C7, R14 (analog Tatser) 03.06.20: Added R26 (Pull Down für TX) 29.07.20: Added Prg_Boot jumper 30.07.20: Added C8, C9, R27 (analog Taster) - Removed LocoNet - Removed CV read option - Added Selextrix OP and connectors - Added opt power supply terminal - Added 5V step down regulator - CAN connector could be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"
- note removed: "Revision History: 31.08.20: - Corrected the LED PCBs (Ver. 1.5 was totaly wrong) - swaped the Input/Output pins (3-Pin header = Input) - corrected the pin assignement of the 3535 WS2812 18.10.20: - Corrected the output of the last connector 31.10.22: - New size of the LED modules - Additional normaly colosed Solder Jumper 05.11.22: - Moved the Selectrix part to this sheet - Added Loconet componen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"
- note removed: "Selectrix (Loconet) Mini Verteiler"
- note removed: "Selectrix und LocoNet (Seite 2)"
- note removed: "ToDo: - 2 oder 3 CAN Busse z.B. für GBM Übersetzung (Hardi GBM -> Märklin) - CAN Int Pin oder zus. Pin für 2/3 CAN Busse mit Galv. Getrenten CAN Modul - Zweite CS Leitung per Lötjumper für IC4 damit man zwei CAN Busse gleichzeitig verwenden kann (für Tests) - Pin6 von LEDs0 und LEDs 2 Stecker mit Pin6 der Miniverteiler verbinden"
- note removed: "Ver.: 1.8.2"
- note removed: "WS2811/WS2812 LED Ansteuerung DCC, Selectrix, CAN LocoNet"
- note removed: "https://pgahtow.de/w/Loconet"
- note removed: "nu = Not used by Loconet"
- moved on the sheet: IC2A, IC2B, IC3C, IC3D, JP4, R21, R22, R23, R24, R25, R28, SJ_LN1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
