File: Platinen/550-WS2811_Stepper/WS2811_Stepper.brd (EAGLE design)
At the start: 71.4 x 38.7 mm, 50 parts, among them CON1 End SW1, CON2 End SW2, CON3 End SW1H, CON4 STEPPER_CON, CON5 End SW2H, CON6 NEMA17, CON7 LED, IC1 4017N, J10 , M1 BOARD_A4988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

Commit message: Corrected missing 4017 Power Supply
Connections:
- removed net VDD: IC1.16
- removed net VSS: IC1.8
- net +5V: now also IC1.16
- net GND: now also IC1.8
Routing:
- net +5V: track 154.0 -> 176.2 mm
- net GND: track 218.7 -> 223.5 mm
Changed lines of the file:
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@@
 <setting verticaltext="up"/>
 </settings>
-<grid distance="12.5" unitdist="mil" unit="mil" style="lines" multiple="1" display="yes" altdistance="12.5" altunitdist="mil" altunit="mil"/>
+<grid distance="12.5" unitdist="mil" unit="mil" style="lines" multiple="1" display="no" altdistance="12.5" altunitdist="mil" altunit="mil"/>
 <layers>
 <layer number="1" name="Top" color="4" fill="1" visible="yes" active="yes"/>
@@
 <text x="62.23" y="8.89" size="1.016" layer="25" rot="R180">&gt;Ver</text>
 <text x="16.1925" y="19.3675" size="1.016" layer="26" rot="MR0">&gt;Ver</text>
-<text x="26.67" y="1.27" size="1.016" layer="25" rot="R180">&gt;Date</text>
+<text x="26.3525" y="1.27" size="1.016" layer="25" rot="R180">&gt;Date</text>
 <text x="16.1925" y="17.4625" size="1.016" layer="26" rot="MR0">&gt;Date</text>
 <text x="53.34" y="11.7475" size="1.016" layer="26" rot="MR0">https://wiki.mobaledlib.de/p550</text>
@@
 </plain>
 <attributes>
-<attribute name="DATE" value="29.05.21"/>
-<attribute name="VER" value="Ver: 1.0.1"/>
+<attribute name="DATE" value="28.9.23"/>
+<attribute name="VER" value="Ver: 1.1"/>
 </attributes>
 <variantdefs>
@@
 <wire x1="46.9392" y1="3.2766" x2="46.101" y2="2.4384" width="0.4064" layer="1"/>
 <wire x1="46.9392" y1="4.1148" x2="46.9392" y2="3.2766" width="0.4064" layer="1"/>
-<wire x1="52.8066" y1="9.9822" x2="46.9392" y2="4.1148" width="0.4064" layer="1"/>
+<wire x1="52.8066" y1="9.9822" x2="49.82845" y2="7.00405" width="0.4064" layer="1"/>
 <wire x1="53.9242" y1="9.9822" x2="52.8066" y2="9.9822" width="0.4064" layer="1"/>
 <wire x1="36.8808" y1="14.4526" x2="36.83" y2="14.605" width="0.4064" layer="1"/>
@@
 <wire x1="27.1018" y1="6.9088" x2="27.1018" y2="3.556" width="0.4064" layer="1"/>
 <wire x1="27.3812" y1="7.1882" x2="27.1018" y2="6.9088" width="0.4064" layer="1"/>
-<wire x1="27.3812" y1="16.4084" x2="27.3812" y2="7.1882" width="0.4064" layer="1"/>
-<wire x1="26.543" y1="17.2466" x2="27.3812" y2="16.4084" width="0.4064" layer="1"/>
-<wire x1="26.543" y1="18.3642" x2="26.543" y2="17.2466" width="0.4064" layer="1"/>
-<wire x1="31.5722" y1="23.3934" x2="26.543" y2="18.3642" width="0.4064" layer="1"/>
-<wire x1="32.9692" y1="23.3934" x2="31.5722" y2="23.3934" width="0.4064" layer="1"/>
-<wire x1="32.9692" y1="23.3934" x2="33.02" y2="23.495" width="0.4064" layer="1"/>
+<wire x1="27.3812" y1="7.1882" x2="27.3812" y2="13.97" width="0.4064" layer="1"/>
 <wire x1="7.6962" y1="28.575" x2="11.4554" y2="28.575" width="0.4064" layer="1"/>
 <wire x1="7.62" y1="6.985" x2="12.065" y2="2.54" width="0.4064" layer="16"/>
@@
 <wire x1="15.1638" y1="34.3662" x2="15.1638" y2="35.4838" width="0.4064" layer="16"/>
 <wire x1="15.1638" y1="35.4838" x2="17.145" y2="37.465" width="0.4064" layer="16"/>
+<contactref element="IC1" pad="8"/>
+<wire x1="27.3812" y1="13.97" x2="25.4" y2="15.9512" width="0.4064" layer="1"/>
+<wire x1="27.94" y1="23.495" x2="33.02" y2="23.495" width="0.4064" layer="1"/>
+<wire x1="25.4" y1="15.9512" x2="25.4" y2="20.955" width="0.4064" layer="1"/>
+<wire x1="25.4" y1="20.955" x2="27.94" y2="23.495" width="0.4064" layer="1"/>
+<wire x1="46.9392" y1="4.1148" x2="46.9392" y2="6.9342" width="0.4064" layer="1"/>
+<wire x1="46.9392" y1="6.9342" x2="46.99" y2="6.985" width="0.4064" layer="1"/>
+<wire x1="46.99" y1="6.985" x2="47.00905" y2="7.00405" width="0.4064" layer="1"/>
+<wire x1="47.00905" y1="7.00405" x2="49.82845" y2="7.00405" width="0.4064" layer="1"/>
 </signal>
 <signal name="+5V">
@@
 <wire x1="67.945" y1="22.86" x2="66.3575" y2="24.4475" width="0.254" layer="1"/>
 <wire x1="66.3575" y1="24.4475" x2="66.3575" y2="26.9875" width="0.254" layer="1"/>
+<contactref element="IC1" pad="16"/>
+<wire x1="26.6954" y1="17.26446875" x2="26.6954" y2="18.29553125" width="0.4064" layer="1"/>
+<wire x1="33.53553125" y1="22.2504" x2="34.2646" y2="22.97946875" width="0.4064" layer="1"/>
+<wire x1="34.2646" y1="22.97946875" x2="34.2646" y2="24.01053125" width="0.4064" layer="1"/>
+<wire x1="34.2646" y1="24.01053125" x2="33.53553125" y2="24.7396" width="0.4064" layer="1"/>
+<wire x1="29.21" y1="14.605" x2="29.21" y2="14.74986875" width="0.4064" layer="1"/>
+<wire x1="28.6004" y1="24.7396" x2="27.94" y2="25.4" width="0.4064" layer="1"/>
+<wire x1="29.21" y1="14.74986875" x2="26.6954" y2="17.26446875" width="0.4064" layer="1"/>
+<wire x1="33.53553125" y1="24.7396" x2="28.6004" y2="24.7396" width="0.4064" layer="1"/>
+<wire x1="26.6954" y1="18.29553125" x2="30.65026875" y2="22.2504" width="0.4064" layer="1"/>
+<wire x1="30.65026875" y1="22.2504" x2="33.53553125" y2="22.2504" width="0.4064" layer="1"/>
 </signal>
 <signal name="N$27">
@@
 <wire x1="22.9362" y1="24.3078" x2="22.9362" y2="29.591" width="0.2032" layer="1"/>
 </signal>
-<signal name="N$17">
-</signal>
-<signal name="VSS">
-<contactref element="IC1" pad="8"/>
-</signal>
-<signal name="VDD">
-<contactref element="IC1" pad="16"/>
-</signal>
 <signal name="N$19">
 <contactref element="IC1" pad="4"/>
@@
 <wire x1="30.7594" y1="17.8562" x2="28.0924" y2="17.8562" width="0.2032" layer="1"/>
 <wire x1="35.0266" y1="22.1234" x2="30.7594" y2="17.8562" width="0.2032" layer="1"/>
-<wire x1="38.227" y1="22.1234" x2="35.0266" y2="22.1234" width="0.2032" layer="1"/>
+<wire x1="38.227" y1="22.1234" x2="35.56" y2="22.1234" width="0.2032" layer="1"/>
+<wire x1="35.56" y1="22.1234" x2="35.0266" y2="22.1234" width="0.2032" layer="1"/>
 <wire x1="39.2938" y1="21.0566" x2="38.227" y2="22.1234" width="0.2032" layer="1"/>
 <wire x1="28.0924" y1="17.8562" x2="27.94" y2="17.78" width="0.2032" layer="1"/>
 <wire x1="39.2938" y1="21.0566" x2="39.37" y2="20.955" width="0.2032" layer="1"/>
-<wire x1="33.0708" y1="25.146" x2="33.0708" y2="27.813" width="0.2032" layer="1"/>
-<wire x1="35.0266" y1="23.1902" x2="33.0708" y2="25.146" width="0.2032" layer="1"/>
-<wire x1="35.0266" y1="22.1234" x2="35.0266" y2="23.1902" width="0.2032" layer="1"/>
-<wire x1="33.0708" y1="27.813" x2="33.02" y2="27.94" width="0.2032" layer="1"/>
 <contactref element="CON7" pad="2"/>
 <wire x1="58.039" y1="18.4187375" x2="57.1462625" y2="17.526" width="0.2032" layer="16"/>
@@
 <wire x1="65.35276875" y1="28.1559" x2="64.18436875" y2="26.9875" width="0.254" layer="16"/>
 <wire x1="65.405" y1="22.86" x2="65.405" y2="23.86186875" width="0.254" layer="16"/>
+<wire x1="33.6578" y1="26.40813125" x2="34.02813125" y2="26.0378" width="0.2032" layer="1"/>
+<wire x1="33.02" y1="27.94" x2="33.6578" y2="27.3022" width="0.2032" layer="1"/>
+<wire x1="33.6578" y1="27.3022" x2="33.6578" y2="26.40813125" width="0.2032" layer="1"/>
+<wire x1="34.02813125" y1="26.0378" x2="34.2872" y2="26.0378" width="0.2032" layer="1"/>
+<wire x1="34.2872" y1="26.0378" x2="35.56" y2="24.765" width="0.2032" layer="1"/>
+<wire x1="35.56" y1="24.765" x2="35.56" y2="22.1234" width="0.2032" layer="1"/>
 </signal>
 <signal name="N$15">
@@
 </signals>
 <mfgpreviewcolors>
-<mfgpreviewcolor name="soldermaskcolor" color="0xC8000000"/>
+<mfgpreviewcolor name="soldermaskcolor" color="0xC8008000"/>
 <mfgpreviewcolor name="silkscreencolor" color="0xFFFEFEFE"/>
 <mfgpreviewcolor name="backgroundcolor" color="0xFF282828"/>

Commit message: added missing Power-Pins IC1
added missing Power-Pins IC1
Routing:
- net +5V: track 176.2 -> 165.6 mm, vias 3 -> 6
- net GND: track 223.5 -> 218.7 mm
